Commit message: Adding collision files for ati, calib and handle

File: lwr_description/urdf/ati_sensor.urdf.xacro (robot description, xacro)
@@ -32,5 +32,5 @@
 	      <origin xyz="0 0 -0.0488" rpy="0 0 ${-45*M_PI/180.0}" />
 	      <geometry>
-		<mesh filename="package://lwr_description/meshes/ati_sensor/ati_sensor.stl" />
+		<mesh filename="package://lwr_description/meshes/ati_sensor/ati_sensor_collision.stl" />
 	      </geometry>
 	    </collision>

File: lwr_description/urdf/calib_tool.urdf.xacro (robot description, xacro)
@@ -28,5 +28,5 @@
 	      <origin xyz="0 0 0" rpy="0 0 0" />
 	      <geometry>
-		<mesh filename="package://lwr_description/meshes/calib_tool/calib_tool.stl" />
+		<mesh filename="package://lwr_description/meshes/calib_tool/calib_tool_collision.stl" />
 	      </geometry>
 	    </collision>

File: lwr_description/urdf/handle.urdf.xacro (robot description, xacro)
@@ -28,5 +28,5 @@
 	      <origin xyz="0 0 0" rpy="0 0 0" />
 	      <geometry>
-		<mesh filename="package://lwr_description/meshes/handle/handle.stl" />
+		<mesh filename="package://lwr_description/meshes/handle/handle_collision.stl" />
 	      </geometry>
 	    </collision>

Commit message: add simpler mesh + real weights

File: lwr_description/urdf/ati_sensor.urdf.xacro (robot description, xacro)
@@ -15,5 +15,5 @@
 		      rpy="0 0 0" />
 		    <mass
-		      value="0.316951020394394" />
+		      value="0.212" />
 		    <inertia
 		      ixx="4.36061005979496E-05"
@@ -44,4 +44,5 @@
     <child link="ati_link" />
   </joint>
+  <!-- The sensing part of the sensor -->
   <link name="ati_link">
     <inertial>
@@ -61,23 +62,21 @@
     <visual>
       <origin
-        xyz="0 0 0"
+        xyz="0 0 -0.005"
         rpy="0 0 0" />
       <geometry>
-        <mesh
-          filename="package://lwr_description/meshes/ati_sensor/ati_sensor_cylinder.stl" />
+        <cylinder length="0.01" radius="0.03"/>
       </geometry>
       <material
         name="">
         <color
-          rgba="0.792156862745098 0.819607843137255 0.933333333333333 1" />
+          rgba="1.0 0.0 0.0 0.1" />
       </material>
     </visual>
     <collision>
       <origin
-        xyz="0 0 0"
+        xyz="0 0 -0.005"
         rpy="0 0 0" />
       <geometry>
-        <mesh
-          filename="package://lwr_description/meshes/ati_sensor/ati_sensor_cylinder.stl" />
+        <cylinder length="0.01" radius="0.03"/>
       </geometry>
     </collision>

Commit message: fix masses

File: lwr_description/urdf/ati_sensor.urdf.xacro (robot description, xacro)
@@ -15,5 +15,5 @@
 		      rpy="0 0 0" />
 		    <mass
-		      value="0.212" />
+		      value="${138+171+212}" />
 		    <inertia
 		      ixx="4.36061005979496E-05"

File: lwr_description/urdf/calib_tool.urdf.xacro (robot description, xacro)
@@ -7,5 +7,5 @@
 		xyz="-0.00289334578157395 3.88856796242065E-07 -0.00147855262054228"
 		rpy="0 0 0" />
-	      <mass value="0.0304913733578414" />
+	      <mass value="0.034" />
 	      <inertia
 		ixx="8.75764054795742E-06"
@@ -36,5 +36,5 @@
 		rpy="0 0 0"
 		xyz="0.0688 0 ${0.0195-0.0488}" />
-	    <parent link="ati_link" />
+	    <parent link="ati_base_link" />
 	    <child link="calib_link" />
 	  </joint>

File: lwr_description/urdf/handle.urdf.xacro (robot description, xacro)
@@ -7,5 +7,5 @@
 		xyz="-1.05305026599362E-05 0.0306221837161532 0.00261872427259377"
 		rpy="0 0 0" />
-	      <mass value="0.066495361381441" />
+	      <mass value="0.100" />
 	      <inertia
 		ixx="0.000102858534792815"

Commit message: Correction of the collision mesh's position

File: lwr_description/urdf/ati_sensor.urdf.xacro (robot description, xacro)
@@ -32,5 +32,5 @@
 	    </visual>
 	    <collision>
-	      <origin xyz="0 0 -0.0488" rpy="0 0 ${-45*M_PI/180.0}" />
+	      <origin xyz="0 0 -0.045" rpy="0 0 ${-45*M_PI/180.0}" />
 	      <geometry>
 		<mesh filename="package://lwr_description/meshes/ati_sensor/ati_sensor_collision.stl" />
