Commit message: New hook

File: lwr_description/urdf/hook.urdf.xacro (robot description, xacro)
@@ -4,13 +4,13 @@
   	<link name="hook_link">
 			<inertial>
-      	<origin	xyz="-0.0254993845921743 1.38777878078145E-17 0.00542364979744681" rpy="0 0 0" />
+      	<origin	xyz="0.00489979385409813 -1.38777878078145E-17 -0.00448859846302793" rpy="0 0 0" />
 	      <mass value="0.00264337359925226" />
       	<inertia
-		      ixx="1.31229592580266E-06"
-		      ixy="-4.65078567008438E-22"
-		      ixz="-1.73070306938344E-07"
-		      iyy="1.80117298509349E-06"
-		      iyz="2.31978685293435E-22"
-		      izz="4.97471327705407E-07" />
+	    ixx="2.25474425622611E-06"
+	    ixy="0"
+	    ixz="1.97404446084148E-07"
+	    iyy="3.19522431280729E-06"
+       	    iyz="1.23621707785698E-22"
+             izz="9.52568601677036E-07" />
 	    </inertial>
   	  <visual>
@@ -33,7 +33,7 @@
   	</link>
 		<joint name="ati_to_hook_joint" type="fixed">
-		  <origin
-		    xyz="-0.036155 -0.025331 0.0444"
-		    rpy="-3.1416 -9.386E-17 -2.7489" />
+		<origin
+		      xyz="-0.012678 -0.017678 0.0394"
+		      rpy="3.1416 -3.5785E-14 -1.1102E-16" />
 		  <parent
 		    link="ati_link" />
