Commit message: Changing max joint value and closed pose

File: lwr_description/urdf/gripper.urdf.xacro (robot description, xacro)
@@ -96,5 +96,5 @@
 		  <axis
 		    xyz="0 0 1" />
-		 <limit lower="0" upper="1.5708" velocity="10.0" effort="1000" />
+		 <limit lower="0" upper="1.05" velocity="10.0" effort="1000" />
 		</joint>
 		<link

Commit message: Adding a new frame for future grasping

File: lwr_description/urdf/gripper.urdf.xacro (robot description, xacro)
@@ -2,8 +2,14 @@
 <robot xmlns:xacro="http://www.ros.org/wiki/xacro">
 	<xacro:macro name="gripper">
-		<joint name="gripper_base_joint" type="fixed">
-			<origin xyz="0 0 0" rpy="0 0 ${M_PI/4}" />
+	  <joint name="gripper_base_joint" type="fixed">
+	    <origin xyz="0 0 0" rpy="0 0 ${M_PI/4}" />
 	    <parent link="ati_link" />
 	    <child link="gripper_base_link" />
+	  </joint>
+	  <link name="gripper_grasp_link" />
+	  <joint name="gripper_grasp_joint" type="fixed">
+	    <origin xyz="0 0 0.085" rpy="0 0 0" />
+	    <parent link="gripper_base_link" />
+	    <child link="gripper_grasp_link" />
 	  </joint>
 		<link name="gripper_base_link">
