Commit message: move properties out of macro

File: lwr_description/urdf/lwr.urdf.xacro (robot description, xacro)
@@ -3,4 +3,7 @@
       xmlns:controller="http://playerstage.sourceforge.net/gazebo/xmlschema/#controller"
    name="lwr" >
+   <xacro:property name="velocity_scale" value="1.0"/>
+   <xacro:property name="effort_scale" value="1.0"/>
+   <property name="M_PI" value="3.1415926535897931" />
   <xacro:macro name="gazebo_reference" params="name">
     <gazebo reference="${name}">
@@ -22,8 +25,5 @@
     <!--<dynamics damping="5.5" friction="1"/>-->
   </xacro:macro>
-   <xacro:property name="velocity_scale" value="1.0"/>
-   <xacro:property name="effort_scale" value="1.0"/>
    <xacro:macro name="lwr" params="parent name prefix *origin ">
-      <property name="M_PI" value="3.1415926535897931" />
       <!-- joint between {parent} and arm_0_link -->
       <joint name="${prefix}/${parent}_base" type="fixed">

Commit message: fix KRL offset

File: lwr_description/urdf/lwr.urdf.xacro (robot description, xacro)
@@ -89,10 +89,10 @@
          <limit lower="${-170 * M_PI / 180}" upper="${170 * M_PI / 180}" effort="${effort_scale * 200}" velocity="${velocity_scale * 112.5 * M_PI / 180}" />
          <dynamics friction="0.0" damping="1.0"/>
-         <origin xyz="0 0 0.103" rpy="0 0 0" />
+         <origin xyz="0 0 0.11" rpy="0 0 0" />
          <axis xyz="0 0 1" />
       </joint>
       <link name="${prefix}/${name}_1_link">
          <inertial>
-            <origin xyz="2.1826998880744087e-05 -0.021623840412335664 -0.07915171924289198" rpy="0.239538165056 0.00537995201801 0.0492155584082" />
+            <origin xyz="0.00021826998880744087 -0.021623840412335664 -0.07915171924289198" rpy="0.239538165056 0.00537995201801 0.0492155584082" />
             <mass value="2.0" />
             <inertia ixx="0.0129545076394" ixy="0" ixz="0" iyy="0.0128178432409" iyz="0" izz="0.00442072765916" />
@@ -146,5 +146,5 @@
          <limit lower="${-120 * M_PI / 180}" upper="${120 * M_PI / 180}" effort="${effort_scale * 200}" velocity="${velocity_scale * 112.5 * M_PI / 180}" />
          <dynamics friction="0.0" damping="1.0"/>
-         <origin xyz="0 0 0.2105" rpy="0 0 0" />
+         <origin xyz="0 0 0.2" rpy="0 0 0" />
          <axis xyz="0 -1 0" />
       </joint>
@@ -186,5 +186,5 @@
          <limit lower="${-170 * M_PI / 180}" upper="${170 * M_PI / 180}" effort="${effort_scale * 100}" velocity="${velocity_scale * 112.5 * M_PI / 180}" />
          <dynamics friction="0.0" damping="1.0"/>
-         <origin xyz="0 0 0.192" rpy="0 0 0" />
+         <origin xyz="0 0 0.2" rpy="0 0 0" />
          <axis xyz="0 0 1" />
       </joint>
@@ -243,5 +243,5 @@
          <limit lower="${-120 * M_PI / 180}" upper="${120 * M_PI / 180}" effort="${effort_scale * 100}" velocity="${velocity_scale * 112.5 * M_PI / 180}" />
          <dynamics friction="0.0" damping="1.0"/>
-         <origin xyz="0 0.003 0.21" rpy="0 0 0" />
+         <origin xyz="0 0.0 0.2" rpy="0 0 0" />
          <axis xyz="0 1 0" />
       </joint>
@@ -300,5 +300,5 @@
          <limit lower="${-170 * M_PI / 180}" upper="${170 * M_PI / 180}" effort="${effort_scale * 100}" velocity="${velocity_scale * 180.0 * M_PI / 180}" />
          <dynamics friction="0.0" damping="1.0"/>
-         <origin xyz="0 0 0.193" rpy="0 0 0" />
+         <origin xyz="0 0 0.2" rpy="0 0 0" />
          <axis xyz="0 0 1" />
       </joint>
@@ -357,5 +357,5 @@
          <limit lower="${-120 * M_PI / 180}" upper="${120 * M_PI / 180}" effort="${effort_scale * 30}" velocity="${velocity_scale * 112.5 * M_PI / 180}" />
          <dynamics friction="0.0" damping="1.0"/>
-         <origin xyz="0 0 0.2" rpy="0 0 0" />
+         <origin xyz="0 0 0.19" rpy="0 0 0" />
          <axis xyz="0 -1 0" />
       </joint>
@@ -414,5 +414,5 @@
          <limit lower="${-170 * M_PI / 180}" upper="${170 * M_PI / 180}" effort="${effort_scale * 30}" velocity="${velocity_scale * 112.5 * M_PI / 180}" />
          <dynamics friction="0.0" damping="1.0"/>
-         <origin xyz="0 0 0.079" rpy="0 0 0" />
+         <origin xyz="0 0 0.078" rpy="0 0 0" />
          <axis xyz="0 0 1" />
       </joint>

Commit message: add inertias from solidworks

File: lwr_description/urdf/lwr.urdf.xacro (robot description, xacro)
@@ -3,7 +3,15 @@
       xmlns:controller="http://playerstage.sourceforge.net/gazebo/xmlschema/#controller"
    name="lwr" >
-   <xacro:property name="velocity_scale" value="1.0"/>
-   <xacro:property name="effort_scale" value="1.0"/>
+   <xacro:property name="velocity_scale" value="20.0"/>
+   <xacro:property name="effort_scale" value="20.0"/>
    <xacro:property name="M_PI" value="3.1415926535897931" />
+   <xacro:property name="damping_factor" value="0.5"/>
+   <xacro:property name="d0" value="${damping_factor*1.0}"/>
+   <xacro:property name="d1" value="${damping_factor*1.0}"/>
+   <xacro:property name="d2" value="${damping_factor*0.5}"/>
+   <xacro:property name="d3" value="${damping_factor*0.5}"/>
+   <xacro:property name="d4" value="${damping_factor*0.5}"/>
+   <xacro:property name="d5" value="${damping_factor*0.1}"/>
+   <xacro:property name="d6" value="${damping_factor*0.1}"/>
   <xacro:macro name="gazebo_reference" params="name">
     <gazebo reference="${name}">
@@ -19,5 +27,5 @@
   <xacro:macro name="gz_joint">
     <provideFeedback>true</provideFeedback>
-    <implicitSpringDamper>true</implicitSpringDamper>
+    <!--implicitSpringDamper>true</implicitSpringDamper-->
     <!--<kp>0.0</kp>[> CFM <]-->
     <!--<kd>0.0</kd>[> ERP <]-->
@@ -26,5 +34,5 @@
   </xacro:macro>
    <xacro:macro name="lwr" params="parent name prefix *origin ">
-      <!-- joint between {parent} and arm_0_link -->
+      <!-- joint between {parent} and lwr_0_link -->
       <joint name="${prefix}/${parent}_base" type="fixed">
         <gazebo reference="${prefix}/${parent}_base">
@@ -36,9 +44,18 @@
       </joint>
       <link name="${prefix}/${name}_0_link">
-         <inertial>
-            <origin xyz="0 0 0" rpy="0 0 0" />
-            <mass value="3.65" />
-            <inertia ixx="0.00805112828804" ixy="0" ixz="0" iyy="0.00845152236845" iyz="0" izz="0.00863585824764" />
-         </inertial>
+          <inertial>
+            <origin
+              xyz="-0.000638499331014356 5.02538509694617E-06 0.0482289968116927"
+              rpy="0 0 0" />
+            <mass
+              value="1.21032454350876" />
+            <inertia
+              ixx="0.00262560565710656"
+              ixy="-5.2754950052563E-07"
+              ixz="3.77940202490646E-05"
+              iyy="0.00280724642508563"
+              iyz="-2.56972470148208E-07"
+              izz="0.00306998250407766" />
+          </inertial>
          <visual>
             <origin xyz="0 0 0" rpy="0 0 ${M_PI}" />
@@ -53,32 +70,7 @@
                <mesh filename="package://lwr_description/meshes/lwr/link0.dae" />
             </geometry>
-           <surface>
-            <friction>
-              <ode>
-                <mu>0.998000</mu>
-                <mu2>0.998000</mu2>
-                <fdir1>0.000000 0.000000 0.000000</fdir1>
-                <slip1>0.000000</slip1>
-                <slip2>0.000000</slip2>
-              </ode>
-            </friction>
-            <bounce>
-              <restitution_coefficient>0.000000</restitution_coefficient>
-              <threshold>100000.000000</threshold>
-            </bounce>
-            <contact>
-              <ode>
-                <soft_cfm>0.000000</soft_cfm>
-                <soft_erp>0.200000</soft_erp>
-                <kp>100000.000000</kp>
-                <kd>1.000000</kd>
-                <max_vel>100.000000</max_vel>
-                <min_depth>0.001000</min_depth>
-              </ode>
-            </contact>
-          </surface>
-         </collision>
-      </link>
-      <!-- joint between arm_0_link and arm_1_link -->
+         </collision>
+      </link>
+      <!-- joint between lwr_0_link and lwr_1_link -->
       <joint name="${prefix}/${name}_0_joint" type="revolute">
         <gazebo reference="${prefix}/${name}_0_joint">
@@ -88,14 +80,23 @@
          <child link="${prefix}/${name}_1_link" />
          <limit lower="${-170 * M_PI / 180}" upper="${170 * M_PI / 180}" effort="${effort_scale * 200}" velocity="${velocity_scale * 112.5 * M_PI / 180}" />
-         <dynamics friction="0.0" damping="1.0"/>
-         <origin xyz="0 0 0.11" rpy="0 0 0" />
+         <dynamics friction="0" damping="${d0}"/>
+         <origin xyz="0 0 0.102" rpy="0 0 0" />
          <axis xyz="0 0 1" />
       </joint>
       <link name="${prefix}/${name}_1_link">
-         <inertial>
-            <origin xyz="0.00021826998880744087 -0.021623840412335664 -0.07915171924289198" rpy="0.239538165056 0.00537995201801 0.0492155584082" />
-            <mass value="2.0" />
-            <inertia ixx="0.0129545076394" ixy="0" ixz="0" iyy="0.0128178432409" iyz="0" izz="0.00442072765916" />
-         </inertial>
+          <inertial>
+            <origin
+              xyz="-6.33965437334127E-08 0.0233273473346096 0.118146290406178"
+              rpy="0 0 0" />
+            <mass
+              value="2.30339938771869" />
+            <inertia
+              ixx="0.0156081163626041"
+              ixy="5.97319920503909E-08"
+              ixz="-1.64780770629425E-07"
+              iyy="0.0153467542173805"
+              iyz="0.00319168949093809"
+              izz="0.00440736079943446" />
+          </inertial>
          <visual>
             <origin xyz="0 0 0" rpy="0 0 ${M_PI}" />
@@ -110,32 +111,7 @@
                <mesh filename="package://lwr_description/meshes/lwr/link1.dae" />
             </geometry>
-           <surface>
-            <friction>
-              <ode>
-                <mu>0.998000</mu>
-                <mu2>0.998000</mu2>
-                <fdir1>0.000000 0.000000 0.000000</fdir1>
-                <slip1>0.000000</slip1>
-                <slip2>0.000000</slip2>
-              </ode>
-            </friction>
-            <bounce>
-              <restitution_coefficient>0.000000</restitution_coefficient>
-              <threshold>100000.000000</threshold>
-            </bounce>
-            <contact>
-              <ode>
-                <soft_cfm>0.000000</soft_cfm>
-                <soft_erp>0.200000</soft_erp>
-                <kp>100000.000000</kp>
-                <kd>1.000000</kd>
-                <max_vel>100.000000</max_vel>
-                <min_depth>0.001000</min_depth>
-              </ode>
-            </contact>
-          </surface>
-         </collision>
-      </link>
-      <!-- joint between arm_1_link and arm_2_link -->
+         </collision>
+      </link>
+      <!-- joint between lwr_1_link and lwr_2_link -->
       <joint name="${prefix}/${name}_1_joint" type="revolute">
         <gazebo reference="${prefix}/${name}_1_joint">
@@ -145,14 +121,23 @@
          <child link="${prefix}/${name}_2_link" />
          <limit lower="${-120 * M_PI / 180}" upper="${120 * M_PI / 180}" effort="${effort_scale * 200}" velocity="${velocity_scale * 112.5 * M_PI / 180}" />
-         <dynamics friction="0.0" damping="1.0"/>
-         <origin xyz="0 0 0.2" rpy="0 0 0" />
+         <dynamics friction="0" damping="${d1}"/>
+         <origin xyz="0 0.0 0.2085" rpy="0 0 0" />
          <axis xyz="0 -1 0" />
       </joint>
       <link name="${prefix}/${name}_2_link">
-         <inertial>
-            <origin xyz="-0.0010097053542516513 0.028478464648332931 0.082033627936009448" rpy="0.252444092172 -0.0167820344187 0.0575928285281" />
-            <mass value="2.0" />
-            <inertia ixx="0.0132950018592" ixy="0" ixz="0" iyy="0.0131003199685" iyz="0" izz="0.0044657387969" />
-         </inertial>
+    <inertial>
+      <origin
+        xyz="1.26774962153076E-06 -0.032746486541291 0.0736556727355962"
+        rpy="0 0 0" />
+      <mass
+        value="2.30343543179071" />
+      <inertia
+        ixx="0.0142348526057094"
+        ixy="-3.73763310100809E-08"
+        ixz="1.70703603169075E-07"
+        iyy="0.0141319978448755"
+        iyz="0.00228090337255746"
+        izz="0.00424792208583136" />
+    </inertial>
          <visual>
             <origin xyz="0 0 0" rpy="0 0 ${M_PI}" />
@@ -177,5 +162,5 @@
          </collision>
       </link>
-      <!-- joint between arm_2_link and arm_3_link -->
+      <!-- joint between lwr_2_link and lwr_3_link -->
       <joint name="${prefix}/${name}_2_joint" type="revolute">
         <gazebo reference="${prefix}/${name}_2_joint">
@@ -185,14 +170,23 @@
          <child link="${prefix}/${name}_3_link" />
          <limit lower="${-170 * M_PI / 180}" upper="${170 * M_PI / 180}" effort="${effort_scale * 100}" velocity="${velocity_scale * 112.5 * M_PI / 180}" />
-         <dynamics friction="0.0" damping="1.0"/>
-         <origin xyz="0 0 0.2" rpy="0 0 0" />
+         <dynamics friction="0" damping="${d2}"/>
+         <origin xyz="0 0 0.1915" rpy="0 0 0" />
          <axis xyz="0 0 1" />
       </joint>
       <link name="${prefix}/${name}_3_link">
-         <inertial>
-            <origin xyz="-0.00068512472584392442 0.022787627643261723 -0.078806475454300237" rpy="-0.211279484805 -0.0186487662306 -0.00721347462905" />
-            <mass value="2.0" />
-            <inertia ixx="0.0127763513867" ixy="0" ixz="0" iyy="0.0128011372133" iyz="0" izz="0.0043627376553" />
-         </inertial>
+    <inertial>
+      <origin
+        xyz="-1.40921289121243E-06 -0.0233297626126898 0.11815047247629"
+        rpy="0 0 0" />
+      <mass
+        value="2.30342143971329" />
+      <inertia
+        ixx="0.0156098024078732"
+        ixy="4.75479645197283E-08"
+        ixz="1.17852233217589E-07"
+        iyy="0.0153476851366831"
+        iyz="-0.00319215869825882"
+        izz="0.0044071430916942" />
+    </inertial>
          <visual>
             <origin xyz="0 0 0" rpy="0 0 ${M_PI}" />
@@ -207,32 +201,7 @@
                <mesh filename="package://lwr_description/meshes/lwr/link3.dae" />
             </geometry>
-           <surface>
-            <friction>
-              <ode>
-                <mu>0.998000</mu>
-                <mu2>0.998000</mu2>
-                <fdir1>0.000000 0.000000 0.000000</fdir1>
-                <slip1>0.000000</slip1>
-                <slip2>0.000000</slip2>
-              </ode>
-            </friction>
-            <bounce>
-              <restitution_coefficient>0.000000</restitution_coefficient>
-              <threshold>100000.000000</threshold>
-            </bounce>
-            <contact>
-              <ode>
-                <soft_cfm>0.000000</soft_cfm>
-                <soft_erp>0.200000</soft_erp>
-                <kp>100000.000000</kp>
-                <kd>1.000000</kd>
-                <max_vel>100.000000</max_vel>
-                <min_depth>0.001000</min_depth>
-              </ode>
-            </contact>
-          </surface>
-         </collision>
-      </link>
-      <!-- joint between arm_3_link and arm_4_link -->
+         </collision>
+      </link>
+      <!-- joint between lwr_3_link and lwr_4_link -->
       <joint name="${prefix}/${name}_3_joint" type="revolute">
         <gazebo reference="${prefix}/${name}_3_joint">
@@ -242,14 +211,23 @@
          <child link="${prefix}/${name}_4_link" />
          <limit lower="${-120 * M_PI / 180}" upper="${120 * M_PI / 180}" effort="${effort_scale * 100}" velocity="${velocity_scale * 112.5 * M_PI / 180}" />
-         <dynamics friction="0.0" damping="1.0"/>
-         <origin xyz="0 0.0 0.2" rpy="0 0 0" />
+         <dynamics friction="0" damping="${d3}"/>
+         <origin xyz="0 0 0.2085" rpy="0 0 0" />
          <axis xyz="0 1 0" />
       </joint>
       <link name="${prefix}/${name}_4_link">
-         <inertial>
-            <origin xyz="-0.00025120620404353643 0.027040543208881447 0.082599870266635594" rpy="0.259090664398 -0.00225330262131 0.0469419954367" />
-            <mass value="2.0" />
-            <inertia ixx="0.0132276730313" ixy="0" ixz="0" iyy="0.0130734228464" iyz="0" izz="0.00439977729281" />
-         </inertial>
+    <inertial>
+      <origin
+        xyz="1.12239473548659E-07 0.0327442387470235 0.073658815701594"
+        rpy="0 0 0" />
+      <mass
+        value="2.30343586527606" />
+      <inertia
+        ixx="0.0142336552604204"
+        ixy="-5.89296043886227E-08"
+        ixz="-1.568273589226E-07"
+        iyy="0.0141315528954361"
+        iyz="-0.00228056254422505"
+        izz="0.00424816761410708" />
+    </inertial>
          <visual>
             <origin xyz="0 0 0" rpy="0 0 ${M_PI}" />
@@ -264,32 +242,7 @@
                <mesh filename="package://lwr_description/meshes/lwr/link4.dae" />
             </geometry>
-           <surface>
-            <friction>
-              <ode>
-                <mu>0.998000</mu>
-                <mu2>0.998000</mu2>
-                <fdir1>0.000000 0.000000 0.000000</fdir1>
-                <slip1>0.000000</slip1>
-                <slip2>0.000000</slip2>
-              </ode>
-            </friction>
-            <bounce>
-              <restitution_coefficient>0.000000</restitution_coefficient>
-              <threshold>100000.000000</threshold>
-            </bounce>
-            <contact>
-              <ode>
-                <soft_cfm>0.000000</soft_cfm>
-                <soft_erp>0.200000</soft_erp>
-                <kp>100000.000000</kp>
-                <kd>1.000000</kd>
-                <max_vel>100.000000</max_vel>
-                <min_depth>0.001000</min_depth>
-              </ode>
-            </contact>
-          </surface>
-         </collision>
-      </link>
-      <!-- joint between arm_4_link and arm_5_link -->
+         </collision>
+      </link>
+      <!-- joint between lwr_4_link and lwr_5_link -->
       <joint name="${prefix}/${name}_4_joint" type="revolute">
         <gazebo reference="${prefix}/${name}_4_joint">
@@ -299,14 +252,23 @@
          <child link="${prefix}/${name}_5_link" />
          <limit lower="${-170 * M_PI / 180}" upper="${170 * M_PI / 180}" effort="${effort_scale * 100}" velocity="${velocity_scale * 180.0 * M_PI / 180}" />
-         <dynamics friction="0.0" damping="1.0"/>
-         <origin xyz="0 0 0.2" rpy="0 0 0" />
+         <dynamics friction="0" damping="${d4}"/>
+         <origin xyz="0 0.0 0.1915" rpy="0 0 0" />
          <axis xyz="0 0 1" />
       </joint>
       <link name="${prefix}/${name}_5_link">
-         <inertial>
-            <origin xyz="-7.2951660343995983e-05 0.034300558520003806 -0.082836449419419589" rpy="-0.399346437469 -0.0238815557936 0.011018430381" />
-            <mass value="2.0" />
-            <inertia ixx="0.0124407882151" ixy="0" ixz="0" iyy="0.0124710412724" iyz="0" izz="0.00438005667842" />
-         </inertial>
+    <inertial>
+      <origin
+        xyz="-6.00824789920296E-07 0.0207751869661564 0.0862053948486382"
+        rpy="0 0 0" />
+      <mass
+        value="1.60059828363332" />
+      <inertia
+        ixx="0.00880806620496216"
+        ixy="1.22820321842462E-07"
+        ixz="-5.66844221164893E-08"
+        iyy="0.00813520145401624"
+        iyz="0.00261443543508601"
+        izz="0.00359712267754715" />
+    </inertial>
          <visual>
             <origin xyz="0 0 0" rpy="0 0 ${M_PI}" />
@@ -321,32 +283,7 @@
                <mesh filename="package://lwr_description/meshes/lwr/link5.dae" />
             </geometry>
-           <surface>
-            <friction>
-              <ode>
-                <mu>0.998000</mu>
-                <mu2>0.998000</mu2>
-                <fdir1>0.000000 0.000000 0.000000</fdir1>
-                <slip1>0.000000</slip1>
-                <slip2>0.000000</slip2>
-              </ode>
-            </friction>
-            <bounce>
-              <restitution_coefficient>0.000000</restitution_coefficient>
-              <threshold>100000.000000</threshold>
-            </bounce>
-            <contact>
-              <ode>
-                <soft_cfm>0.000000</soft_cfm>
-                <soft_erp>0.200000</soft_erp>
-                <kp>100000.000000</kp>
-                <kd>1.000000</kd>
-                <max_vel>100.000000</max_vel>
-                <min_depth>0.001000</min_depth>
-              </ode>
-            </contact>
-          </surface>
-         </collision>
-      </link>
-      <!-- joint between arm_5_link and arm_6_link -->
+         </collision>
+      </link>
+      <!-- joint between lwr_5_link and lwr_6_link -->
       <joint name="${prefix}/${name}_5_joint" type="revolute">
         <gazebo reference="${prefix}/${name}_5_joint">
@@ -356,14 +293,23 @@
          <child link="${prefix}/${name}_6_link" />
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
Commit message: Enhance damping

File: lwr_description/urdf/lwr.urdf.xacro (robot description, xacro)
@@ -3,14 +3,14 @@
       xmlns:controller="http://playerstage.sourceforge.net/gazebo/xmlschema/#controller"
    name="lwr" >
-   <xacro:property name="velocity_scale" value="20.0"/>
-   <xacro:property name="effort_scale" value="20.0"/>
+   <xacro:property name="velocity_scale" value="50.0"/>
+   <xacro:property name="effort_scale" value="50.0"/>
    <xacro:property name="M_PI" value="3.1415926535897931" />
-   <xacro:property name="damping_factor" value="0.5"/>
-   <xacro:property name="d0" value="${damping_factor*1.0}"/>
-   <xacro:property name="d1" value="${damping_factor*1.0}"/>
-   <xacro:property name="d2" value="${damping_factor*0.5}"/>
-   <xacro:property name="d3" value="${damping_factor*0.5}"/>
-   <xacro:property name="d4" value="${damping_factor*0.5}"/>
-   <xacro:property name="d5" value="${damping_factor*0.1}"/>
+   <xacro:property name="damping_factor" value="1.0"/>
+   <xacro:property name="d0" value="${damping_factor*5.5}"/>
+   <xacro:property name="d1" value="${damping_factor*5.5}"/>
+   <xacro:property name="d2" value="${damping_factor*3.5}"/>
+   <xacro:property name="d3" value="${damping_factor*3.5}"/>
+   <xacro:property name="d4" value="${damping_factor*3.5}"/>
+   <xacro:property name="d5" value="${damping_factor*1.1}"/>
    <xacro:property name="d6" value="${damping_factor*0.1}"/>
   <xacro:macro name="gazebo_reference" params="name">
