Commit message: removes unnecessary gazebo stuff

File: lwr_description/urdf/lwr.urdf.xacro (robot description, xacro)
@@ -15,18 +15,7 @@
    <xacro:property name="d6" value="${damping_factor*0.1}"/>
   <!-- Gazebo joint configuration -->
-  <xacro:macro  name="gz_joint">
-    <provideFeedback>true</provideFeedback>
-    <!--implicitSpringDamper>true</implicitSpringDamper-->
-    <!--<kp>0.0</kp>[> CFM <]-->
-    <!--<kd>0.0</kd>[> ERP <]-->
-    <!--<cfmDamping>true</cfmDamping>-->
-    <!--<dynamics damping="5.5" friction="1"/>-->
-  </xacro:macro>
    <xacro:macro name="lwr" params="parent *origin ">
       <!-- joint between {parent} and lwr_0_link -->
       <joint name="joint_base" type="fixed">
-        <gazebo reference="joint_base">
-          <xacro:gz_joint/>
-        </gazebo>
          <xacro:insert_block name="origin" />
          <parent link="${parent}" />
@@ -64,7 +53,4 @@
       <!-- joint between lwr_0_link and lwr_1_link -->
       <joint name="joint_0" type="revolute">
-        <gazebo reference="joint_0">
-          <xacro:gz_joint/>
-        </gazebo>
          <parent link="link_0" />
          <child link="link_1" />
@@ -105,7 +91,4 @@
       <!-- joint between lwr_1_link and lwr_2_link -->
       <joint name="joint_1" type="revolute">
-        <gazebo reference="joint_1">
-          <xacro:gz_joint/>
-        </gazebo>
          <parent link="link_1" />
          <child link="link_2" />
@@ -154,7 +137,4 @@
       <!-- joint between lwr_2_link and lwr_3_link -->
       <joint name="joint_2" type="revolute">
-        <gazebo reference="joint_2">
-          <xacro:gz_joint/>
-        </gazebo>
          <parent link="link_2" />
          <child link="link_3" />
@@ -195,7 +175,4 @@
       <!-- joint between lwr_3_link and lwr_4_link -->
       <joint name="joint_3" type="revolute">
-        <gazebo reference="joint_3">
-          <xacro:gz_joint/>
-        </gazebo>
          <parent link="link_3" />
          <child link="link_4" />
@@ -236,7 +213,4 @@
       <!-- joint between lwr_4_link and lwr_5_link -->
       <joint name="joint_4" type="revolute">
-        <gazebo reference="joint_4">
-          <xacro:gz_joint/>
-        </gazebo>
          <parent link="link_4" />
          <child link="link_5" />
@@ -277,7 +251,4 @@
       <!-- joint between lwr_5_link and lwr_6_link -->
       <joint name="joint_5" type="revolute">
-        <gazebo reference="joint_5">
-          <xacro:gz_joint/>
-        </gazebo>
          <parent link="link_5" />
          <child link="link_6" />
@@ -318,7 +289,4 @@
       <!-- joint between lwr_6_link and lwr_7_link -->
       <joint name="joint_6" type="revolute">
-        <gazebo reference="joint_6">
-          <xacro:gz_joint/>
-        </gazebo>
          <parent link="link_6" />
          <child link="link_7" />

Commit message: Add simplifed and very simplified (c2) collision meshes

File: lwr_description/urdf/lwr.urdf.xacro (robot description, xacro)
@@ -47,5 +47,5 @@
             <origin xyz="0 0 0" rpy="0 0 ${M_PI}" />
             <geometry>
-               <mesh filename="package://lwr_description/meshes/lwr/link0.dae" />
+               <mesh filename="package://lwr_description/meshes/lwr/link0_c2.stl" />
             </geometry>
          </collision>
@@ -85,5 +85,5 @@
             <origin xyz="0 0 0" rpy="0 0 ${M_PI}" />
             <geometry>
-               <mesh filename="package://lwr_description/meshes/lwr/link1.dae" />
+               <mesh filename="package://lwr_description/meshes/lwr/link1_c2.stl" />
             </geometry>
          </collision>
@@ -123,5 +123,5 @@
             <origin xyz="0 0 0" rpy="0 0 ${M_PI}" />
             <geometry>
-               <mesh filename="package://lwr_description/meshes/lwr/link2.dae" />
+               <mesh filename="package://lwr_description/meshes/lwr/link2_c2.stl" />
             </geometry>
            <surface>
@@ -169,5 +169,5 @@
             <origin xyz="0 0 0" rpy="0 0 ${M_PI}" />
             <geometry>
-               <mesh filename="package://lwr_description/meshes/lwr/link3.dae" />
+               <mesh filename="package://lwr_description/meshes/lwr/link3_c2.stl" />
             </geometry>
          </collision>
@@ -207,5 +207,5 @@
             <origin xyz="0 0 0" rpy="0 0 ${M_PI}" />
             <geometry>
-               <mesh filename="package://lwr_description/meshes/lwr/link4.dae" />
+               <mesh filename="package://lwr_description/meshes/lwr/link4_c2.stl" />
             </geometry>
          </collision>
@@ -245,5 +245,5 @@
             <origin xyz="0 0 0" rpy="0 0 ${M_PI}" />
             <geometry>
-               <mesh filename="package://lwr_description/meshes/lwr/link5.dae" />
+               <mesh filename="package://lwr_description/meshes/lwr/link5_c2.stl" />
             </geometry>
          </collision>
@@ -283,5 +283,5 @@
             <origin xyz="0 0 0" rpy="0 0 ${M_PI}" />
             <geometry>
-               <mesh filename="package://lwr_description/meshes/lwr/link6.dae" />
+               <mesh filename="package://lwr_description/meshes/lwr/link6_c2.stl" />
             </geometry>
          </collision>
@@ -321,5 +321,5 @@
             <origin xyz="0 0 0" rpy="0 0 ${M_PI}" />
             <geometry>
-               <mesh filename="package://lwr_description/meshes/lwr/link7.dae" />
+               <mesh filename="package://lwr_description/meshes/lwr/link7_c2.stl" />
             </geometry>
          </collision>

Commit message: add friction (Coulomb)

File: lwr_description/urdf/lwr.urdf.xacro (robot description, xacro)
@@ -6,5 +6,5 @@
    <xacro:property name="effort_scale" value="50.0"/>
    <xacro:property name="M_PI" value="3.1415926535897931" />
-   <xacro:property name="damping_factor" value="1.0"/>
+   <xacro:property name="damping_factor" value="0.2"/>
    <xacro:property name="d0" value="${damping_factor*5.5}"/>
    <xacro:property name="d1" value="${damping_factor*5.5}"/>
@@ -14,4 +14,12 @@
    <xacro:property name="d5" value="${damping_factor*1.1}"/>
    <xacro:property name="d6" value="${damping_factor*0.1}"/>
+   <xacro:property name="friction_factor" value="2.0"/>
+   <xacro:property name="f0" value="${friction_factor*1.0}"/>
+   <xacro:property name="f1" value="${friction_factor*1.0}"/>
+   <xacro:property name="f2" value="${friction_factor*1.0}"/>
+   <xacro:property name="f3" value="${friction_factor*1.0}"/>
+   <xacro:property name="f4" value="${friction_factor*1.0}"/>
+   <xacro:property name="f5" value="${friction_factor*1.0}"/>
+   <xacro:property name="f6" value="${friction_factor*1.0}"/>
   <!-- Gazebo joint configuration -->
    <xacro:macro name="lwr" params="parent *origin ">
@@ -56,5 +64,5 @@
          <child link="link_1" />
          <limit lower="${-170 * M_PI / 180}" upper="${170 * M_PI / 180}" effort="${effort_scale * 200}" velocity="${velocity_scale * 112.5 * M_PI / 180}" />
-         <dynamics friction="0" damping="${d0}"/>
+         <dynamics friction="${f0}" damping="${d0}"/>
          <origin xyz="0 0 0.102" rpy="0 0 0" />
          <axis xyz="0 0 1" />
@@ -94,5 +102,5 @@
          <child link="link_2" />
          <limit lower="${-120 * M_PI / 180}" upper="${120 * M_PI / 180}" effort="${effort_scale * 200}" velocity="${velocity_scale * 112.5 * M_PI / 180}" />
-         <dynamics friction="0" damping="${d1}"/>
+         <dynamics friction="${f1}" damping="${d1}"/>
          <origin xyz="0 0.0 0.2085" rpy="0 0 0" />
          <axis xyz="0 -1 0" />
@@ -140,5 +148,5 @@
          <child link="link_3" />
          <limit lower="${-170 * M_PI / 180}" upper="${170 * M_PI / 180}" effort="${effort_scale * 100}" velocity="${velocity_scale * 112.5 * M_PI / 180}" />
-         <dynamics friction="0" damping="${d2}"/>
+         <dynamics friction="${f2}" damping="${d2}"/>
          <origin xyz="0 0 0.1915" rpy="0 0 0" />
          <axis xyz="0 0 1" />
@@ -178,5 +186,5 @@
          <child link="link_4" />
          <limit lower="${-120 * M_PI / 180}" upper="${120 * M_PI / 180}" effort="${effort_scale * 100}" velocity="${velocity_scale * 112.5 * M_PI / 180}" />
-         <dynamics friction="0" damping="${d3}"/>
+         <dynamics friction="${f3}" damping="${d3}"/>
          <origin xyz="0 0 0.2085" rpy="0 0 0" />
          <axis xyz="0 1 0" />
@@ -216,5 +224,5 @@
          <child link="link_5" />
          <limit lower="${-170 * M_PI / 180}" upper="${170 * M_PI / 180}" effort="${effort_scale * 100}" velocity="${velocity_scale * 180.0 * M_PI / 180}" />
-         <dynamics friction="0" damping="${d4}"/>
+         <dynamics friction="${f4}" damping="${d4}"/>
          <origin xyz="0 0.0 0.1915" rpy="0 0 0" />
          <axis xyz="0 0 1" />
@@ -254,5 +262,5 @@
          <child link="link_6" />
          <limit lower="${-120 * M_PI / 180}" upper="${120 * M_PI / 180}" effort="${effort_scale * 30}" velocity="${velocity_scale * 112.5 * M_PI / 180}" />
-         <dynamics friction="0" damping="${d5}"/>
+         <dynamics friction="${f5}" damping="${d5}"/>
          <origin xyz="0 0 0.1985" rpy="0 0 0" />
          <axis xyz="0 -1 0" />
@@ -292,5 +300,5 @@
          <child link="link_7" />
          <limit lower="${-170 * M_PI / 180}" upper="${170 * M_PI / 180}" effort="${effort_scale * 30}" velocity="${velocity_scale * 112.5 * M_PI / 180}" />
-         <dynamics friction="0" damping="${d6}"/>
+         <dynamics friction="${f6}" damping="${d6}"/>
          <origin xyz="0 0 0.078" rpy="0 0 0" />
          <axis xyz="0 0 1" />

Commit message: New damping and Frictions values (OK with moveit)

File: lwr_description/urdf/lwr.urdf.xacro (robot description, xacro)
@@ -3,24 +3,23 @@
       xmlns:controller="http://playerstage.sourceforge.net/gazebo/xmlschema/#controller"
    name="lwr" >
-   <xacro:property name="velocity_scale" value="50.0"/>
+   <xacro:property name="velocity_scale" value="1.0"/>
    <xacro:property name="effort_scale" value="50.0"/>
    <xacro:property name="M_PI" value="3.1415926535897931" />
-   <xacro:property name="damping_factor" value="0.2"/>
-   <xacro:property name="d0" value="${damping_factor*5.5}"/>
-   <xacro:property name="d1" value="${damping_factor*5.5}"/>
-   <xacro:property name="d2" value="${damping_factor*3.5}"/>
-   <xacro:property name="d3" value="${damping_factor*3.5}"/>
-   <xacro:property name="d4" value="${damping_factor*3.5}"/>
-   <xacro:property name="d5" value="${damping_factor*1.1}"/>
-   <xacro:property name="d6" value="${damping_factor*0.1}"/>
-   <xacro:property name="friction_factor" value="2.0"/>
+   <xacro:property name="damping_factor" value="0.1"/>
+   <xacro:property name="d0" value="${damping_factor*2.0}"/>
+   <xacro:property name="d1" value="${damping_factor*1.8}"/>
+   <xacro:property name="d2" value="${damping_factor*1.0}"/>
+   <xacro:property name="d3" value="${damping_factor*1.5}"/>
+   <xacro:property name="d4" value="${damping_factor*1.2}"/>
+   <xacro:property name="d5" value="${damping_factor*1.0}"/>
+   <xacro:property name="d6" value="${damping_factor*1.0}"/>
+   <xacro:property name="friction_factor" value="1.0"/>
    <xacro:property name="f0" value="${friction_factor*1.0}"/>
    <xacro:property name="f1" value="${friction_factor*1.0}"/>
    <xacro:property name="f2" value="${friction_factor*1.0}"/>
    <xacro:property name="f3" value="${friction_factor*1.0}"/>
-   <xacro:property name="f4" value="${friction_factor*1.0}"/>
-   <xacro:property name="f5" value="${friction_factor*1.0}"/>
-   <xacro:property name="f6" value="${friction_factor*1.0}"/>
-  <!-- Gazebo joint configuration -->
+   <xacro:property name="f4" value="${friction_factor*0.4}"/>
+   <xacro:property name="f5" value="${friction_factor*0.1}"/>
+   <xacro:property name="f6" value="${friction_factor*0.1}"/>
    <xacro:macro name="lwr" params="parent *origin ">
       <!-- joint between {parent} and lwr_0_link -->
@@ -73,6 +72,6 @@
               xyz="-6.33965437334127E-08 0.0233273473346096 0.118146290406178"
               rpy="0 0 0" />
-            <mass
-              value="2.30339938771869" />
+              <mass
+                value="2.30339938771869" />
             <inertia
               ixx="0.0156081163626041"
@@ -111,6 +110,6 @@
         xyz="1.26774962153076E-06 -0.032746486541291 0.0736556727355962"
         rpy="0 0 0" />
-      <mass
-        value="2.30343543179071" />
+        <mass
+          value="2.30343543179071" />
       <inertia
         ixx="0.0142348526057094"
@@ -157,6 +156,6 @@
         xyz="-1.40921289121243E-06 -0.0233297626126898 0.11815047247629"
         rpy="0 0 0" />
-      <mass
-        value="2.30342143971329" />
+        <mass
+          value="2.30342143971329" />
       <inertia
         ixx="0.0156098024078732"
@@ -195,6 +194,6 @@
         xyz="1.12239473548659E-07 0.0327442387470235 0.073658815701594"
         rpy="0 0 0" />
-      <mass
-        value="2.30343586527606" />
+        <mass
+          value="2.30343586527606" />
       <inertia
         ixx="0.0142336552604204"
@@ -233,6 +232,6 @@
         xyz="-6.00824789920296E-07 0.0207751869661564 0.0862053948486382"
         rpy="0 0 0" />
-      <mass
-        value="1.60059828363332" />
+        <mass
+          value="1.60059828363332" />
       <inertia
         ixx="0.00880806620496216"
@@ -271,13 +270,13 @@
         xyz="-2.64519244286276E-08 -0.00451753627467652 -0.00295324741635017"
         rpy="0 0 0" />
-      <mass
-        value="1.49302436988808" />
-      <inertia
-        ixx="0.00298541138330797"
-        ixy="-3.97658663154265E-09"
-        ixz="-1.71667243685877E-09"
-        iyy="0.00299834927882566"
-        iyz="-2.53647350791604E-05"
-        izz="0.00323627047307316" />
+        <mass
+          value="1.49302436988808" />
+        <inertia
+          ixx="0.00298541138330797"
+          ixy="-3.97658663154265E-09"
+          ixz="-1.71667243685877E-09"
+          iyy="0.00299834927882566"
+          iyz="-2.53647350791604E-05"
+          izz="0.00323627047307316" />
     </inertial>
          <visual>
@@ -309,13 +308,13 @@
         xyz="2.77555756156289E-17 1.11022302462516E-16 -0.015814675599801"
         rpy="0 0 0" />
-      <mass
-        value="0.108688241139613" />
-      <inertia
-        ixx="4.17908737998876E-05"
-        ixy="0"
-        ixz="0"
-        iyy="4.17908737998876E-05"
-        iyz="0"
-        izz="7.00756879151782E-05" />
+        <mass
+          value="0.108688241139613" />
+        <inertia
+          ixx="4.17908737998876E-05"
+          ixy="0"
+          ixz="0"
+          iyy="4.17908737998876E-05"
+          iyz="0"
+          izz="7.00756879151782E-05" />
     </inertial>
          <visual>

Commit message: velocity scale back to 1.0

File: lwr_description/urdf/lwr.urdf.xacro (robot description, xacro)
@@ -4,5 +4,5 @@
    name="lwr" >
    <xacro:property name="velocity_scale" value="1.0"/>
-   <xacro:property name="effort_scale" value="50.0"/>
+   <xacro:property name="effort_scale" value="1.0"/>
    <xacro:property name="M_PI" value="3.1415926535897931" />
    <xacro:property name="damping_factor" value="0.1"/>

Commit message: test high higher inertias

File: lwr_description/urdf/lwr.urdf.xacro (robot description, xacro)
@@ -4,5 +4,5 @@
    name="lwr" >
    <xacro:property name="velocity_scale" value="1.0"/>
-   <xacro:property name="effort_scale" value="1.0"/>
+   <xacro:property name="effort_scale" value="10.0"/>
    <xacro:property name="M_PI" value="3.1415926535897931" />
    <xacro:property name="damping_factor" value="0.1"/>
@@ -37,10 +37,10 @@
               value="1.21032454350876" />
             <inertia
-              ixx="0.00262560565710656"
+              ixx="0.0262560565710656"
               ixy="-5.2754950052563E-07"
               ixz="3.77940202490646E-05"
-              iyy="0.00280724642508563"
+              iyy="0.0280724642508563"
               iyz="-2.56972470148208E-07"
-              izz="0.00306998250407766" />
+              izz="0.0306998250407766" />
           </inertial>
          <visual>
@@ -75,10 +75,10 @@
                 value="2.30339938771869" />
             <inertia
-              ixx="0.0156081163626041"
+              ixx="0.156081163626041"
               ixy="5.97319920503909E-08"
               ixz="-1.64780770629425E-07"
-              iyy="0.0153467542173805"
-              iyz="0.00319168949093809"
-              izz="0.00440736079943446" />
+              iyy="0.153467542173805"
+              iyz="0.0319168949093809"
+              izz="0.0440736079943446" />
           </inertial>
          <visual>
@@ -273,10 +273,10 @@
           value="1.49302436988808" />
         <inertia
-          ixx="0.00298541138330797"
+          ixx="0.0298541138330797"
           ixy="-3.97658663154265E-09"
           ixz="-1.71667243685877E-09"
-          iyy="0.00299834927882566"
+          iyy="0.0299834927882566"
           iyz="-2.53647350791604E-05"
-          izz="0.00323627047307316" />
+          izz="0.0323627047307316" />
     </inertial>
          <visual>
@@ -311,10 +311,10 @@
           value="0.108688241139613" />
         <inertia
-          ixx="4.17908737998876E-05"
+          ixx="4.17908737998876E-02"
           ixy="0"
           ixz="0"
-          iyy="4.17908737998876E-05"
+          iyy="4.17908737998876E-02"
           iyz="0"
-          izz="7.00756879151782E-05" />
+          izz="7.00756879151782E-02" />
     </inertial>
          <visual>

Commit message: Alternate joint_names for Anis

File: lwr_description/urdf/lwr.urdf.xacro (robot description, xacro)
@@ -59,5 +59,5 @@
       </link>
       <!-- joint between lwr_0_link and lwr_1_link -->
-      <joint name="joint_0" type="revolute">
+      <joint name="lbr4_j0" type="revolute">
          <parent link="link_0" />
          <child link="link_1" />
@@ -97,5 +97,5 @@
       </link>
       <!-- joint between lwr_1_link and lwr_2_link -->
-      <joint name="joint_1" type="revolute">
+      <joint name="lbr4_j1" type="revolute">
          <parent link="link_1" />
          <child link="link_2" />
@@ -143,5 +143,5 @@
       </link>
       <!-- joint between lwr_2_link and lwr_3_link -->
-      <joint name="joint_2" type="revolute">
+      <joint name="lbr4_j2" type="revolute">
          <parent link="link_2" />
          <child link="link_3" />
@@ -181,5 +181,5 @@
       </link>
       <!-- joint between lwr_3_link and lwr_4_link -->
-      <joint name="joint_3" type="revolute">
+      <joint name="lbr4_j3" type="revolute">
          <parent link="link_3" />
          <child link="link_4" />
@@ -219,5 +219,5 @@
       </link>
       <!-- joint between lwr_4_link and lwr_5_link -->
-      <joint name="joint_4" type="revolute">
+      <joint name="lbr4_j4" type="revolute">
          <parent link="link_4" />
          <child link="link_5" />
@@ -257,5 +257,5 @@
       </link>
       <!-- joint between lwr_5_link and lwr_6_link -->
-      <joint name="joint_5" type="revolute">
+      <joint name="lbr4_j5" type="revolute">
          <parent link="link_5" />
          <child link="link_6" />
@@ -295,5 +295,5 @@
       </link>
       <!-- joint between lwr_6_link and lwr_7_link -->
-      <joint name="joint_6" type="revolute">
+      <joint name="lbr4_j6" type="revolute">
          <parent link="link_6" />
          <child link="link_7" />
