Commit message: Fix table inertia and weight

File: lwr_description/urdf/table.urdf.xacro (robot description, xacro)
@@ -3,4 +3,9 @@
    <xacro:macro name="table">
 	  <link name="table_link">
+      <inertial>
+        <origin xyz="0 0 0" rpy="0 0 0"/>
+        <mass value="200"/>
+        <inertia ixx="0.1"  ixy="0"  ixz="0" iyy="0.1" iyz="0" izz="0.1" />
+      </inertial>
 	    <visual>
 	      <origin xyz="0 0 0" rpy="-1.5707963267948966 0 0" />

Commit message: Remove textures on table .dae loading fails with realtime_urdf_filter

File: lwr_description/urdf/table.urdf.xacro (robot description, xacro)
@@ -9,8 +9,11 @@
       </inertial>
 	    <visual>
-	      <origin xyz="0 0 0" rpy="-1.5707963267948966 0 0" />
+ 	      <origin xyz="0 0 0" rpy="0 0 0" />
 	      <geometry>
-		        <mesh filename="package://lwr_description/meshes/table/table.dae" />
+		        <mesh filename="package://lwr_description/meshes/table/table.stl" />
 	      </geometry>
+	      <material name="table_color">
+		      <color rgba="${210/255} ${170/255} ${120/255} 1.0"/>
+      	</material>
 	    </visual>
 	    <collision>
