Commit message: Fix inertia for camera -- rviz visu

File: lwr_description/urdf/head_cam.urdf.xacro (robot description, xacro)
@@ -6,5 +6,5 @@
         <origin xyz="0 0 0.5" rpy="0 0 0"/>
         <mass value="0.1"/>
-        <inertia ixx="10"  ixy="0"  ixz="0" iyy="10" iyz="0" izz="10" />
+        <inertia ixx="0.001"  ixy="0"  ixz="0" iyy="0.001" iyz="0" izz="0.001" />
       </inertial>
       <visual>

Commit message: Fix camera collision

File: lwr_description/urdf/head_cam.urdf.xacro (robot description, xacro)
@@ -18,5 +18,5 @@
       </visual>
       <collision>
-        <origin xyz="0 0 0" rpy="0 0 0"/>
+        <origin xyz="${-0.045/2.0} 0 0" rpy="0 0 0"/>
         <geometry>
           <box size="0.045 0.042 0.032" />

Commit message: Simulate epingle

File: lwr_description/urdf/head_cam.urdf.xacro (robot description, xacro)
@@ -1,8 +1,48 @@
 <?xml version="1.0" encoding="UTF-8"?>
 <robot xmlns:xacro="http://www.ros.org/wiki/xacro">
+   <xacro:property name="epingle_length" value="0.09" />
+   <xacro:property name="epingle_radius" value="0.002" />
+   <xacro:property name="motor_length" value="0.02" />
+   <xacro:property name="motor_radius" value="0.025" />
    <xacro:macro name="head_cam">
+     <link name="epingle_link" >
+       <inertial>
+         <origin xyz="0 0 0.5" rpy="0 0 0"/>
+         <mass value="0.1"/>
+         <inertia ixx="0.001"  ixy="0"  ixz="0" iyy="0.001" iyz="0" izz="0.001" />
+       </inertial>
+       <visual name="motor">
+         <origin xyz="0 0 0" rpy="0 0 0" />
+         <geometry>
+           <cylinder length="${motor_length}" radius="${motor_radius}" />
+         </geometry>
+       </visual>
+       <visual name="epingle">
+         <origin xyz="0 0 ${epingle_length/2.0}" rpy="0 0 0" />
+         <geometry>
+           <cylinder length="${epingle_length}" radius="${epingle_radius}" />
+         </geometry>
+       </visual>
+       <collision name="motor_collision">
+         <origin xyz="0 0 0" rpy="0 0 0" />
+         <geometry>
+           <cylinder length="${motor_length}" radius="${motor_radius}" />
+         </geometry>
+       </collision>
+       <collision name="epingle_collision">
+         <origin xyz="0 0 ${epingle_length/2.0}" rpy="0 0 0" />
+         <geometry>
+           <cylinder length="${epingle_length}" radius="${epingle_radius}" />
+         </geometry>
+      </collision>
+    </link>
+    <joint name="epingle_joint" type="fixed">
+      <origin xyz="0 0 ${motor_length/2.0}" rpy="0 0 0"/>
+      <parent link="ati_link"/>
+      <child link="epingle_link"/>
+    </joint>
 	  <link name="cam_link" >
       <inertial>
-        <origin xyz="0 0 0.5" rpy="0 0 0"/>
+        <origin xyz="${-0.045/2.0} ${-0.042/2.0} ${-0.032/2.0}" rpy="0 0 0"/>
         <mass value="0.1"/>
         <inertia ixx="0.001"  ixy="0"  ixz="0" iyy="0.001" iyz="0" izz="0.001" />
@@ -24,6 +64,13 @@
       </collision>
 	  </link>
+    <link name="epingle_tip_link" />
+    <joint name="ati_to_tip_joint" type="fixed">
+      <origin rpy="${M_PI} 0 0" xyz="0 0 ${motor_length+epingle_length}" />
+	    <parent link="ati_link" />
+	    <child link="epingle_tip_link" />
+	  </joint>
 	  <joint name="ati_to_cam_joint" type="fixed">
-	    <origin rpy="3.141592 -0.46 3.141592" xyz="0.1 0 0" />
+	    <!--origin rpy="${M_PI} ${-M_PI/2.0+atan(0.1/(motor_length+epingle_length))} ${M_PI}" xyz="0.1 0 0" /-->
+      	<origin rpy="${M_PI} -0.8329812666744316 ${M_PI}" xyz="0.1 0 0" />
 	    <parent link="ati_link" />
 	    <child link="cam_link" />

Commit message: Correct head_cam_link

File: lwr_description/urdf/head_cam.urdf.xacro (robot description, xacro)
@@ -4,13 +4,13 @@
     <link name="head_cam_link">
       <inertial>
-        <origin xyz="-0.001317 0.032906 -0.0621" rpy="0 0 0" />
-        <mass value="0.23396" />
+        <origin xyz="-0.0621004664004336 -0.00131697898890089 0.0329063947179623" rpy="0 0 0" />
+        <mass value="0.233958232943254" />
         <inertia
-          ixx="0.00047366"
-          ixy="-5.9303E-07"
-          ixz="1.6112E-06"
-          iyy="0.00016812"
-          iyz="-1.0497E-05"
-          izz="0.00043559" />
+          ixx="0.000435587148701726"
+          ixy="1.6112175747291E-06"
+          ixz="-1.04965927091446E-05"
+          iyy="0.000473661487000832"
+          iyz="-5.93028607241656E-07"
+          izz="0.000168118719518926" />
       </inertial>
       <visual>
@@ -20,5 +20,5 @@
         </geometry>
         <material name="">
-          <color rgba="0.49804 0.49804 0.49804 1" />
+          <color rgba="0.498039215686275 0.498039215686275 0.498039215686275 1" />
         </material>
       </visual>
@@ -31,10 +31,10 @@
     </link>
     <joint name="ati_to_cam_joint" type="fixed">
-        <origin
-          xyz="0.00138820343559641 -0.113248229330811 0.053096412734154"
-          rpy="-0.436332312998576 8.73838564895237E-16 3.05311331771918E-15" />
-        <parent link="ati_link" />
-        <child link="head_cam_link" />
-        <axis xyz="0 0 0" />
+      <origin
+        xyz="0.00138820343559641 -0.113248229330811 0.053096412734154"
+        rpy="-3.14159265358979 -1.13446401379632 1.5707963267949" />
+      <parent link="ati_link" />
+      <child link="head_cam_link" />
+      <axis xyz="0 0 0" />
     </joint>
     <link name="head_cam_link_optical" />

Commit message: Fixing bad assembly of parts

File: lwr_description/urdf/head_cam.urdf.xacro (robot description, xacro)
@@ -4,13 +4,13 @@
     <link name="head_cam_link">
       <inertial>
-        <origin xyz="-0.0621004664004336 -0.00131697898890089 0.0329063947179623" rpy="0 0 0" />
+        <origin xyz="-0.0621004664004336 -0.00186849655878642 0.0329063947179623" rpy="0 0 0" />
         <mass value="0.233958232943254" />
         <inertia
-          ixx="0.000435587148701726"
-          ixy="1.6112175747291E-06"
-          ixz="-1.04965927091446E-05"
+          ixx="0.000435876167618103"
+          ixy="2.30524748763368E-06"
+          ixz="-1.04965927091447E-05"
           iyy="0.000473661487000832"
-          iyz="-5.93028607241656E-07"
-          izz="0.000168118719518926" />
+          iyz="-4.07790014097315E-06"
+          izz="0.000168407738435303" />
       </inertial>
       <visual>
@@ -32,5 +32,5 @@
     <joint name="ati_to_cam_joint" type="fixed">
       <origin
-        xyz="0.00138820343559641 -0.113248229330811 0.053096412734154"
+        xyz="0.00238820343559641 -0.113248229330811 0.053096412734154"
         rpy="-3.14159265358979 -1.13446401379632 1.5707963267949" />
       <parent link="ati_link" />

File: lwr_description/urdf/screwdriver.urdf.xacro (robot description, xacro)
@@ -5,14 +5,14 @@
       <inertial>
         <origin
-          xyz="6.93889390390723E-18 6.93889390390723E-18 -0.0710432844406097"
+          xyz="-2.08166817117217E-17 -1.38777878078145E-17 -0.0728518735920298"
           rpy="0 0 0" />
-        <mass value="0.122887323635982" />
+        <mass value="0.123766969578987" />
         <inertia
-          ixx="0.000154793314803634"
+          ixx="0.000168714135052911"
           ixy="0"
-          ixz="-4.966674522813E-21"
-          iyy="0.000154793314803634"
-          iyz="9.10679255368707E-21"
-          izz="3.48079006878619E-05" />
+          ixz="-5.18908039078516E-20"
+          iyy="0.000168714135052911"
+          iyz="-5.87098767652812E-21"
+          izz="3.49811909386339E-05" />
       </inertial>
       <visual>
@@ -34,5 +34,5 @@
     <joint name="ati_to_screwdriver_joint" type="fixed">
       <origin
-        xyz="0 0 0.11"
+        xyz="0 0 0.115"
         rpy="-4.6259E-16 9.0159E-16 9.992E-16" />
       <parent link="ati_link" />

Commit message: New meshes for screwdriver and head_cam

File: lwr_description/urdf/head_cam.urdf.xacro (robot description, xacro)
@@ -4,13 +4,13 @@
     <link name="head_cam_link">
       <inertial>
-        <origin xyz="-0.0621004664004336 -0.00186849655878642 0.0329063947179623" rpy="0 0 0" />
-        <mass value="0.233958232943254" />
+        <origin xyz="-0.00025044 -1.1935E-15 -0.0028882" rpy="0 0 0" />
+        <mass value="0.036942" />
         <inertia
-          ixx="0.000435876167618103"
-          ixy="2.30524748763368E-06"
-          ixz="-1.04965927091447E-05"
-          iyy="0.000473661487000832"
-          iyz="-4.07790014097315E-06"
-          izz="0.000168407738435303" />
+          ixx="9.1578E-06"
+          ixy="-1.207E-20"
+          ixz="-8.1587E-10"
+          iyy="8.8696E-06"
+          iyz="-8.61E-22"
+          izz="1.7832E-05" />
       </inertial>
       <visual>
@@ -32,6 +32,6 @@
     <joint name="ati_to_cam_joint" type="fixed">
       <origin
-        xyz="0.0023882 -0.11747 0.044033"
-        rpy="-3.1416 -1.1345 1.5708" />
+        xyz="0.0023882 -0.12154 0.044879"
+        rpy="-3.1416 -1.1781 1.5708" />
       <parent link="ati_link" />
       <child link="head_cam_link" />

File: lwr_description/urdf/screwdriver.urdf.xacro (robot description, xacro)
@@ -5,14 +5,14 @@
       <inertial>
         <origin
-          xyz="-2.08166817117217E-17 -1.38777878078145E-17 -0.0728518735920298"
+          xyz="0.00019306 -0.00063333 -0.10165"
           rpy="0 0 0" />
-        <mass value="0.123766969578987" />
+        <mass value="0.22973" />
         <inertia
-          ixx="0.000168714135052911"
-          ixy="0"
-          ixz="-5.18908039078516E-20"
-          iyy="0.000168714135052911"
-          iyz="-5.87098767652812E-21"
-          izz="3.49811909386339E-05" />
+          ixx="0.00044365"
+          ixy="2.5405E-07"
+          ixz="-1.8342E-06"
+          iyy="0.00044758"
+          iyz="5.3828E-06"
+          izz="0.00010303" />
       </inertial>
       <visual>
@@ -34,5 +34,5 @@
     <joint name="ati_to_screwdriver_joint" type="fixed">
       <origin
-        xyz="0 0 0.115"
+        xyz="0 0 0.16"
         rpy="-4.6259E-16 9.0159E-16 9.992E-16" />
       <parent link="ati_link" />
