Commit message: add fake limits

File: lwr_description/urdf/calib_tool.urdf.xacro (robot description, xacro)
@@ -38,4 +38,5 @@
 	    <parent link="ati_base_link" />
 	    <child link="calib_link" />
+        <limit effort="400" velocity="0" lower="0" upper="0" />
 	  </joint>
    </xacro:macro>

File: lwr_description/urdf/handle.urdf.xacro (robot description, xacro)
@@ -38,4 +38,5 @@
 	    <parent link="ati_base_link" />
 	    <child link="handle_link" />
+        <limit effort="400" velocity="0" lower="0" upper="0" />
 	  </joint>
    </xacro:macro>

File: lwr_description/urdf/head_cam.urdf.xacro (robot description, xacro)
@@ -37,4 +37,5 @@
       <child link="head_cam_link" />
       <axis xyz="0 0 0" />
+      <limit effort="400" velocity="0" lower="0" upper="0" />
     </joint>
     <link name="head_cam_link_optical" />
@@ -46,4 +47,5 @@
       <parent link="head_cam_link"/>
       <child link="head_cam_link_optical"/>
+      <limit effort="400" velocity="0" lower="0" upper="0" />
     </joint>
   </xacro:macro>

File: lwr_description/urdf/hook.urdf.xacro (robot description, xacro)
@@ -41,4 +41,5 @@
 		    link="hook_link" />
 		  <axis xyz="0 0 0" />
+          <limit effort="400" velocity="0" lower="0" upper="0" />
 		</joint>
   </xacro:macro>

File: lwr_description/urdf/screwdriver.urdf.xacro (robot description, xacro)
@@ -39,4 +39,5 @@
       <child link="screwdriver_link" />
       <axis xyz="0 0 1" />
+      <limit effort="400" velocity="0" lower="0" upper="0" />
     </joint>
   </xacro:macro>

File: lwr_description/urdf/table.urdf.xacro (robot description, xacro)
@@ -25,4 +25,5 @@
 	    <parent link="table_link" />
 	    <child link="base_link" />
+        <limit effort="40000" velocity="0" lower="0" upper="0" />
 	  </joint>
    </xacro:macro>

Commit message: New position of the calib tool on the ati sensor

File: lwr_description/urdf/calib_tool.urdf.xacro (robot description, xacro)
@@ -34,7 +34,7 @@
 	  <joint name="ati_to_calib_joint" type="fixed">
 	    <origin
-		rpy="0 0 0"
-		xyz="0.0688 0 ${0.0195-0.0488}" />
-	    <parent link="ati_base_link" />
+		rpy="0 0 -1.5708"
+		xyz="0 -0.0688 ${0.02-0.0488}" />
+	    <parent link="ati_link" />
 	    <child link="calib_link" />
         <limit effort="400" velocity="0" lower="0" upper="0" />
