Commit message: handle is now attached to base ati

File: lwr_description/urdf/handle.urdf.xacro (robot description, xacro)
@@ -34,7 +34,7 @@
 	  <joint name="ati_to_handle_joint" type="fixed">
 	    <origin
-	      xyz="0 0.0438 ${0.0075-0.0488}"
+	      xyz="0 0.0438 -0.0375"
 	      rpy="0 0 0" />
-	    <parent link="ati_link" />
+	    <parent link="ati_base_link" />
 	    <child link="handle_link" />
 	  </joint>

Commit message: New handle and camera mesh and position

File: lwr_description/urdf/handle.urdf.xacro (robot description, xacro)
@@ -34,6 +34,6 @@
 	  <joint name="ati_to_handle_joint" type="fixed">
 	    <origin
-	      xyz="0 0.0438 -0.0375"
-	      rpy="0 0 0" />
+	      xyz="${cos(3*pi/4)*0.0438} ${sin(3*pi/4)*0.0438} -0.035"
+	      rpy="0 0 ${pi/4}" />
 	    <parent link="ati_base_link" />
 	    <child link="handle_link" />

File: lwr_description/urdf/head_cam.urdf.xacro (robot description, xacro)
@@ -32,7 +32,7 @@
     <joint name="ati_to_cam_joint" type="fixed">
       <origin
-        xyz="0.0023882 -0.12154 0.044879"
-        rpy="-3.1416 -1.1781 1.5708" />
-      <parent link="ati_link" />
+        xyz="${-cos(3*pi/4)*0.0438} ${-sin(3*pi/4)*0.0438} -0.0375"
+        rpy="0 0 ${5*pi/4}" />
+      <parent link="ati_base_link" />
       <child link="head_cam_link" />
       <axis xyz="0 0 0" />
@@ -44,5 +44,5 @@
           image won't be aligned properly with the frame it is supposedly
           originating from -->
-      <origin xyz="0 0 0" rpy="-1.570796 0 -1.570796"/>
+      <origin xyz="0 0 0" rpy="${-pi/2} 0 ${-pi/2}"/>
       <parent link="head_cam_link"/>
       <child link="head_cam_link_optical"/>
