Commit message: fix spawn_urdf crash on indigo

File: lwr_description/gazebo/lwr.gazebo.urdf.xacro (robot description, xacro)
@@ -1,14 +1,8 @@
 <?xml version="1.0"?>
 <robot xmlns:xacro="http://ros.org/wiki/xacro">
-			<!--plugin name="gazebo_ros_moveit_planning_scene" filename="libgazebo_ros_moveit_planning_scene.so">
-			    <robotNamespace>~</robotNamespace>
-			    <sceneName>B08</sceneName>
-			    <robotName>lwr</robotName>
-			    <updatePeriod>0.033</updatePeriod>
-			    <topicName>planning_scene</topicName>
-    		</plugin-->
 	<xacro:macro name="lwr_gazebo" params="name prefix">
 		<gazebo>
 			<plugin name="rtt_gazebo" filename="librtt_gazebo_deployer.so">
+				<robotNamespace>~</robotNamespace>
 			  <component>
 			    <package>rtt_lwr_gazebo</package>
@@ -17,5 +11,4 @@
 			  </component>
 			    <orocosScript><filename>$(arg ops_script)</filename></orocosScript>
-			    <!--luaScript><filename>$(arg lua_script)</filename></luaScript-->
 			</plugin>
   		</gazebo>

File: lwr_description/urdf/lwr.urdf.xacro (robot description, xacro)
@@ -5,5 +5,5 @@
    <xacro:property name="velocity_scale" value="1.0"/>
    <xacro:property name="effort_scale" value="1.0"/>
-   <property name="M_PI" value="3.1415926535897931" />
+   <xacro:property name="M_PI" value="3.1415926535897931" />
   <xacro:macro name="gazebo_reference" params="name">
     <gazebo reference="${name}">

Commit message: update link/joint names

File: lwr_description/gazebo/lwr.gazebo.urdf.xacro (robot description, xacro)
@@ -13,33 +13,33 @@
 			</plugin>
   		</gazebo>
-		<gazebo reference="${prefix}/${name}_0_link">
+		<gazebo reference="${prefix}/link_0">
 			<gravity>true</gravity>
 			<material>Gazebo/Orange</material>
 		</gazebo>
-		<gazebo reference="${prefix}/${name}_1_link">
+		<gazebo reference="${prefix}/link_1">
 			<gravity>true</gravity>
 			<material>Gazebo/Orange</material>
 		</gazebo>
-		<gazebo reference="${prefix}/${name}_2_link">
+		<gazebo reference="${prefix}/link_2">
 			<gravity>true</gravity>
 			<material>Gazebo/Orange</material>
 		</gazebo>
-		<gazebo reference="${prefix}/${name}_3_link">
+		<gazebo reference="${prefix}/link_3">
 			<gravity>true</gravity>
 			<material>Gazebo/Orange</material>
 		</gazebo>
-		<gazebo reference="${prefix}/${name}_4_link">
+		<gazebo reference="${prefix}/link_4">
 			<gravity>true</gravity>
 			<material>Gazebo/Orange</material>
 		</gazebo>
-		<gazebo reference="${prefix}/${name}_5_link">
+		<gazebo reference="${prefix}/link_5">
 			<gravity>true</gravity>
 			<material>Gazebo/Orange</material>
 		</gazebo>
-		<gazebo reference="${prefix}/${name}_6_link">
+		<gazebo reference="${prefix}/link_6">
 			<gravity>true</gravity>
 			<material>Gazebo/Grey</material>
 		</gazebo>
-		<gazebo reference="${prefix}/${name}_7_link">
+		<gazebo reference="${prefix}/link_7">
 			<gravity>true</gravity>
 			<material>Gazebo/Grey</material>

File: lwr_description/robots/kuka_lwr.urdf.xacro (robot description, xacro)
@@ -11,24 +11,19 @@
   <!-- materials for visualization -->
   <xacro:include filename="$(find lwr_description)/urdf/materials.urdf.xacro" />
-  <!-- world + base link-->
+  <!-- world-->
   <link name="world"/>
-  <link name="$(arg prefix)/base_link"/>
-  <joint name="$(arg prefix)/base_joint" type="fixed">
-    <parent link="world" />
-    <child link="$(arg prefix)/base_link" />
-  </joint>
-  <gazebo reference="$(arg prefix)/base_link">
+  <gazebo reference="world">
     <static>true</static>>
   </gazebo>
 <xacro:macro name="tool">
-      <link name="$(arg prefix)/kuka_polaris"/>
+      <link name="$(arg prefix)/polaris"/>
       <joint name="$(arg prefix)/tool_joint" type="fixed">
-         <parent link="$(arg prefix)/${name}_7_link" />
-         <child link="$(arg prefix)/kuka_polaris" />
+         <parent link="$(arg prefix)/link_7" />
+         <child link="$(arg prefix)/polaris" />
 	       <origin xyz="0 0 0.055" rpy="0 0 0" />
       </joint>
 </xacro:macro>
   <!--lbr-->
-  <xacro:lwr prefix="$(arg prefix)" name="${name}" parent="$(arg prefix)/base_link">
+  <xacro:lwr prefix="$(arg prefix)" name="${name}" parent="world">
     <!-- Position from origin -->
     <origin xyz="0 0 0.01" rpy="0 0 ${2*M_PI/3}" />

File: lwr_description/urdf/lwr.transmission.xacro (robot description, xacro)
@@ -2,56 +2,56 @@
 <robot xmlns:xacro="http://ros.org/wiki/xacro">
     <xacro:macro name="lwr_transmission" params="name prefix">
-	    <transmission name="${prefix}/${name}_0_trans">
+	    <transmission name="${prefix}/trans_0">
 			<type>transmission_interface/SimpleTransmission</type>
-			<joint name="${prefix}/${name}_0_joint"/>
-			<actuator name="${prefix}/${name}_0_motor">
+			<joint name="${prefix}/joint_0"/>
+			<actuator name="${prefix}/motor_0">
 				<hardwareInterface>EffortJointInterface</hardwareInterface>
 				<mechanicalReduction>1</mechanicalReduction>
 			</actuator>
 	    </transmission>
-		<transmission name="${prefix}/${name}_1_trans">
+		<transmission name="${prefix}/trans_1">
 			<type>transmission_interface/SimpleTransmission</type>
-			<joint name="${prefix}/${name}_1_joint"/>
-			<actuator name="${prefix}/${name}_1_motor">
+			<joint name="${prefix}/joint_1"/>
+			<actuator name="${prefix}/motor_1">
 				<hardwareInterface>EffortJointInterface</hardwareInterface>
 				<mechanicalReduction>1</mechanicalReduction>
 			</actuator>
 		</transmission>
-		<transmission name="${prefix}/${name}_2_trans">
+		<transmission name="${prefix}/trans_2">
 			<type>transmission_interface/SimpleTransmission</type>
-			<joint name="${prefix}/${name}_2_joint"/>
-			<actuator name="${prefix}/${name}_2_motor">
+			<joint name="${prefix}/joint_2"/>
+			<actuator name="${prefix}/motor_2">
 				<hardwareInterface>EffortJointInterface</hardwareInterface>
 				<mechanicalReduction>1</mechanicalReduction>
 			</actuator>
 		</transmission>
-		<transmission name="${prefix}/${name}_3_trans">
+		<transmission name="${prefix}/trans_3">
 			<type>transmission_interface/SimpleTransmission</type>
-			<joint name="${prefix}/${name}_3_joint"/>
-			<actuator name="${prefix}/${name}_3_motor">
+			<joint name="${prefix}/joint_3"/>
+			<actuator name="${prefix}/motor_3">
 				<hardwareInterface>EffortJointInterface</hardwareInterface>
 				<mechanicalReduction>1</mechanicalReduction>
 			</actuator>
 		</transmission>
-		<transmission name="${prefix}/${name}_4_trans">
+		<transmission name="${prefix}/trans_4">
 			<type>transmission_interface/SimpleTransmission</type>
-			<joint name="${prefix}/${name}_4_joint"/>
-			<actuator name="${prefix}/${name}_4_motor">
+			<joint name="${prefix}/joint_4"/>
+			<actuator name="${prefix}/motor_4">
 				<hardwareInterface>EffortJointInterface</hardwareInterface>
 				<mechanicalReduction>1</mechanicalReduction>
 			</actuator>
 		</transmission>
-		<transmission name="${prefix}/${name}_5_trans">
+		<transmission name="${prefix}/trans_5">
 			<type>transmission_interface/SimpleTransmission</type>
-			<joint name="${prefix}/${name}_5_joint"/>
-			<actuator name="${prefix}/${name}_5_motor">
+			<joint name="${prefix}/joint_5"/>
+			<actuator name="${prefix}/motor_5">
 				<hardwareInterface>EffortJointInterface</hardwareInterface>
 				<mechanicalReduction>1</mechanicalReduction>
 			</actuator>
 		</transmission>
-		<transmission name="${prefix}/${name}_6_trans">
+		<transmission name="${prefix}/trans_6">
 			<type>transmission_interface/SimpleTransmission</type>
-			<joint name="${prefix}/${name}_6_joint"/>
-			<actuator name="${prefix}/${name}_6_motor">
+			<joint name="${prefix}/joint_6"/>
+			<actuator name="${prefix}/motor_6">
 				<hardwareInterface>EffortJointInterface</hardwareInterface>
 				<mechanicalReduction>1</mechanicalReduction>

File: lwr_description/urdf/lwr.urdf.xacro (robot description, xacro)
@@ -25,5 +25,5 @@
   </xacro:macro>
   <!-- Gazebo joint configuration -->
-  <xacro:macro name="gz_joint">
+  <xacro:macro  name="gz_joint">
     <provideFeedback>true</provideFeedback>
     <!--implicitSpringDamper>true</implicitSpringDamper-->
@@ -35,13 +35,13 @@
    <xacro:macro name="lwr" params="parent name prefix *origin ">
       <!-- joint between {parent} and lwr_0_link -->
-      <joint name="${prefix}/${parent}_base" type="fixed">
-        <gazebo reference="${prefix}/${parent}_base">
+      <joint name="${prefix}/joint_base" type="fixed">
+        <gazebo reference="${prefix}/joint_base">
           <xacro:gz_joint/>
         </gazebo>
          <xacro:insert_block name="origin" />
          <parent link="${parent}" />
-         <child link="${prefix}/${name}_0_link" />
-      </joint>
-      <link name="${prefix}/${name}_0_link">
+         <child link="${prefix}/link_0" />
+      </joint>
+      <link name="${prefix}/link_0">
           <inertial>
             <origin
@@ -73,10 +73,10 @@
       </link>
       <!-- joint between lwr_0_link and lwr_1_link -->
-      <joint name="${prefix}/${name}_0_joint" type="revolute">
-        <gazebo reference="${prefix}/${name}_0_joint">
-          <xacro:gz_joint/>
-        </gazebo>
-         <parent link="${prefix}/${name}_0_link" />
-         <child link="${prefix}/${name}_1_link" />
+      <joint name="${prefix}/joint_0" type="revolute">
+        <gazebo reference="${prefix}/joint_0">
+          <xacro:gz_joint/>
+        </gazebo>
+         <parent link="${prefix}/link_0" />
+         <child link="${prefix}/link_1" />
          <limit lower="${-170 * M_PI / 180}" upper="${170 * M_PI / 180}" effort="${effort_scale * 200}" velocity="${velocity_scale * 112.5 * M_PI / 180}" />
          <dynamics friction="0" damping="${d0}"/>
@@ -84,5 +84,5 @@
          <axis xyz="0 0 1" />
       </joint>
-      <link name="${prefix}/${name}_1_link">
+      <link name="${prefix}/link_1">
           <inertial>
             <origin
@@ -114,10 +114,10 @@
       </link>
       <!-- joint between lwr_1_link and lwr_2_link -->
-      <joint name="${prefix}/${name}_1_joint" type="revolute">
-        <gazebo reference="${prefix}/${name}_1_joint">
-          <xacro:gz_joint/>
-        </gazebo>
-         <parent link="${prefix}/${name}_1_link" />
-         <child link="${prefix}/${name}_2_link" />
+      <joint name="${prefix}/joint_1" type="revolute">
+        <gazebo reference="${prefix}/joint_1">
+          <xacro:gz_joint/>
+        </gazebo>
+         <parent link="${prefix}/link_1" />
+         <child link="${prefix}/link_2" />
          <limit lower="${-120 * M_PI / 180}" upper="${120 * M_PI / 180}" effort="${effort_scale * 200}" velocity="${velocity_scale * 112.5 * M_PI / 180}" />
          <dynamics friction="0" damping="${d1}"/>
@@ -125,5 +125,5 @@
          <axis xyz="0 -1 0" />
       </joint>
-      <link name="${prefix}/${name}_2_link">
+      <link name="${prefix}/link_2">
     <inertial>
       <origin
@@ -163,10 +163,10 @@
       </link>
       <!-- joint between lwr_2_link and lwr_3_link -->
-      <joint name="${prefix}/${name}_2_joint" type="revolute">
-        <gazebo reference="${prefix}/${name}_2_joint">
-          <xacro:gz_joint/>
-        </gazebo>
-         <parent link="${prefix}/${name}_2_link" />
-         <child link="${prefix}/${name}_3_link" />
+      <joint name="${prefix}/joint_2" type="revolute">
+        <gazebo reference="${prefix}/joint_2">
+          <xacro:gz_joint/>
+        </gazebo>
+         <parent link="${prefix}/link_2" />
+         <child link="${prefix}/link_3" />
          <limit lower="${-170 * M_PI / 180}" upper="${170 * M_PI / 180}" effort="${effort_scale * 100}" velocity="${velocity_scale * 112.5 * M_PI / 180}" />
          <dynamics friction="0" damping="${d2}"/>
@@ -174,5 +174,5 @@
          <axis xyz="0 0 1" />
       </joint>
-      <link name="${prefix}/${name}_3_link">
+      <link name="${prefix}/link_3">
     <inertial>
       <origin
@@ -204,10 +204,10 @@
       </link>
       <!-- joint between lwr_3_link and lwr_4_link -->
-      <joint name="${prefix}/${name}_3_joint" type="revolute">
-        <gazebo reference="${prefix}/${name}_3_joint">
-          <xacro:gz_joint/>
-        </gazebo>
-         <parent link="${prefix}/${name}_3_link" />
-         <child link="${prefix}/${name}_4_link" />
+      <joint name="${prefix}/joint_3" type="revolute">
+        <gazebo reference="${prefix}/joint_3">
+          <xacro:gz_joint/>
+        </gazebo>
+         <parent link="${prefix}/link_3" />
+         <child link="${prefix}/link_4" />
          <limit lower="${-120 * M_PI / 180}" upper="${120 * M_PI / 180}" effort="${effort_scale * 100}" velocity="${velocity_scale * 112.5 * M_PI / 180}" />
          <dynamics friction="0" damping="${d3}"/>
@@ -215,5 +215,5 @@
          <axis xyz="0 1 0" />
       </joint>
-      <link name="${prefix}/${name}_4_link">
+      <link name="${prefix}/link_4">
     <inertial>
       <origin
@@ -245,10 +245,10 @@
       </link>
       <!-- joint between lwr_4_link and lwr_5_link -->
-      <joint name="${prefix}/${name}_4_joint" type="revolute">
-        <gazebo reference="${prefix}/${name}_4_joint">
-          <xacro:gz_joint/>
-        </gazebo>
-         <parent link="${prefix}/${name}_4_link" />
-         <child link="${prefix}/${name}_5_link" />
+      <joint name="${prefix}/joint_4" type="revolute">
+        <gazebo reference="${prefix}/joint_4">
+          <xacro:gz_joint/>
+        </gazebo>
+         <parent link="${prefix}/link_4" />
+         <child link="${prefix}/link_5" />
          <limit lower="${-170 * M_PI / 180}" upper="${170 * M_PI / 180}" effort="${effort_scale * 100}" velocity="${velocity_scale * 180.0 * M_PI / 180}" />
          <dynamics friction="0" damping="${d4}"/>
@@ -256,5 +256,5 @@
          <axis xyz="0 0 1" />
       </joint>
-      <link name="${prefix}/${name}_5_link">
+      <link name="${prefix}/link_5">
     <inertial>
       <origin
@@ -286,10 +286,10 @@
       </link>
       <!-- joint between lwr_5_link and lwr_6_link -->
-      <joint name="${prefix}/${name}_5_joint" type="revolute">
-        <gazebo reference="${prefix}/${name}_5_joint">
-          <xacro:gz_joint/>
-        </gazebo>
-         <parent link="${prefix}/${name}_5_link" />
-         <child link="${prefix}/${name}_6_link" />
+      <joint name="${prefix}/joint_5" type="revolute">
+        <gazebo reference="${prefix}/joint_5">
+          <xacro:gz_joint/>
+        </gazebo>
+         <parent link="${prefix}/link_5" />
+         <child link="${prefix}/link_6" />
          <limit lower="${-120 * M_PI / 180}" upper="${120 * M_PI / 180}" effort="${effort_scale * 30}" velocity="${velocity_scale * 112.5 * M_PI / 180}" />
          <dynamics friction="0" damping="${d5}"/>
@@ -297,5 +297,5 @@
          <axis xyz="0 -1 0" />
       </joint>
-      <link name="${prefix}/${name}_6_link">
+      <link name="${prefix}/link_6">
     <inertial>
       <origin
@@ -327,10 +327,10 @@
       </link>
       <!-- joint between lwr_6_link and lwr_7_link -->
-      <joint name="${prefix}/${name}_6_joint" type="revolute">
-        <gazebo reference="${prefix}/${name}_6_joint">
-          <xacro:gz_joint/>
-        </gazebo>
-         <parent link="${prefix}/${name}_6_link" />
-         <child link="${prefix}/${name}_7_link" />
+      <joint name="${prefix}/joint_6" type="revolute">
+        <gazebo reference="${prefix}/joint_6">
+          <xacro:gz_joint/>
+        </gazebo>
+         <parent link="${prefix}/link_6" />
+         <child link="${prefix}/link_7" />
          <limit lower="${-170 * M_PI / 180}" upper="${170 * M_PI / 180}" effort="${effort_scale * 30}" velocity="${velocity_scale * 112.5 * M_PI / 180}" />
          <dynamics friction="0" damping="${d6}"/>
@@ -338,5 +338,5 @@
          <axis xyz="0 0 1" />
       </joint>
-      <link name="${prefix}/${name}_7_link">
+      <link name="${prefix}/link_7">
     <inertial>
       <origin
@@ -367,6 +367,4 @@
          </collision>
       </link>
-      <!-- Tool macro -->
-      <xacro:tool/>
    </xacro:macro>
 </robot>
