Commit message: Removes prefix (using tf_prefix and namespaces instead)

File: lwr_description/gazebo/lwr.gazebo.urdf.xacro (robot description, xacro)
@@ -1,5 +1,5 @@
 <?xml version="1.0"?>
 <robot xmlns:xacro="http://ros.org/wiki/xacro">
-	<xacro:macro name="lwr_gazebo" params="name prefix">
+	<xacro:macro name="lwr_gazebo">
 		<gazebo>
 			<plugin name="rtt_gazebo" filename="librtt_gazebo_deployer.so">
@@ -10,36 +10,36 @@
 			    <name>lwr_gazebo</name>
 			  </component>
-			    <orocosScript><filename>$(arg ops_script)</filename></orocosScript>
+			    <orocosScript><filename>$(find rtt_lwr_gazebo)/scripts/lwr_gazebo.ops</filename></orocosScript>
 			</plugin>
   		</gazebo>
-		<gazebo reference="${prefix}/link_0">
+		<gazebo reference="link_0">
 			<gravity>true</gravity>
 			<material>Gazebo/Orange</material>
 		</gazebo>
-		<gazebo reference="${prefix}/link_1">
+		<gazebo reference="link_1">
 			<gravity>true</gravity>
 			<material>Gazebo/Orange</material>
 		</gazebo>
-		<gazebo reference="${prefix}/link_2">
+		<gazebo reference="link_2">
 			<gravity>true</gravity>
 			<material>Gazebo/Orange</material>
 		</gazebo>
-		<gazebo reference="${prefix}/link_3">
+		<gazebo reference="link_3">
 			<gravity>true</gravity>
 			<material>Gazebo/Orange</material>
 		</gazebo>
-		<gazebo reference="${prefix}/link_4">
+		<gazebo reference="link_4">
 			<gravity>true</gravity>
 			<material>Gazebo/Orange</material>
 		</gazebo>
-		<gazebo reference="${prefix}/link_5">
+		<gazebo reference="link_5">
 			<gravity>true</gravity>
 			<material>Gazebo/Orange</material>
 		</gazebo>
-		<gazebo reference="${prefix}/link_6">
+		<gazebo reference="link_6">
 			<gravity>true</gravity>
 			<material>Gazebo/Grey</material>
 		</gazebo>
-		<gazebo reference="${prefix}/link_7">
+		<gazebo reference="link_7">
 			<gravity>true</gravity>
 			<material>Gazebo/Grey</material>

File: lwr_description/robots/kuka_lwr.urdf.xacro (robot description, xacro)
@@ -3,5 +3,4 @@
        name="lwr" >
   <property name="M_PI" value="3.1415926535897931" />
-  <property name="name" value="lwr" />
   <!-- lbr-->
   <xacro:include filename="$(find lwr_description)/urdf/lwr.urdf.xacro" />
@@ -13,21 +12,28 @@
   <!-- world-->
   <link name="world"/>
-  <gazebo reference="world">
+  <link name="base_link"/>
+  <joint name="base_joint" type="fixed">
+    <parent link="world"/>
+    <child link="base_link"/>
+    <origin xyz="0 0 0"/>
+  </joint>
+  <gazebo reference="base_link">
     <static>true</static>>
   </gazebo>
-<xacro:macro name="tool">
-      <link name="$(arg prefix)/polaris"/>
-      <joint name="$(arg prefix)/tool_joint" type="fixed">
-         <parent link="$(arg prefix)/link_7" />
-         <child link="$(arg prefix)/polaris" />
-	       <origin xyz="0 0 0.055" rpy="0 0 0" />
-      </joint>
-</xacro:macro>
+  <xacro:macro name="tool">
+    <link name="ati_link"/>
+    <joint name="ati_joint" type="fixed">
+       <parent link="link_7" />
+       <child link="ati_link" />
+       <origin xyz="0 0 0.049" rpy="0 0 0" />
+    </joint>
+  </xacro:macro>
   <!--lbr-->
-  <xacro:lwr prefix="$(arg prefix)" name="${name}" parent="world">
+  <xacro:lwr parent="base_link">
     <!-- Position from origin -->
     <origin xyz="0 0 0.01" rpy="0 0 ${2*M_PI/3}" />
   </xacro:lwr>
-   <xacro:lwr_gazebo prefix="$(arg prefix)" name="${name}"/>
-   <xacro:lwr_transmission prefix="$(arg prefix)" name="${name}"/>
+   <xacro:lwr_gazebo/>
+   <xacro:lwr_transmission/>
+   <xacro:tool/>
 </robot>

File: lwr_description/urdf/lwr.transmission.xacro (robot description, xacro)
@@ -1,57 +1,57 @@
 <?xml version="1.0"?>
 <robot xmlns:xacro="http://ros.org/wiki/xacro">
-    <xacro:macro name="lwr_transmission" params="name prefix">
-	    <transmission name="${prefix}/trans_0">
+    <xacro:macro name="lwr_transmission">
+	    <transmission name="trans_0">
 			<type>transmission_interface/SimpleTransmission</type>
-			<joint name="${prefix}/joint_0"/>
-			<actuator name="${prefix}/motor_0">
+			<joint name="joint_0"/>
+			<actuator name="motor_0">
 				<hardwareInterface>EffortJointInterface</hardwareInterface>
 				<mechanicalReduction>1</mechanicalReduction>
 			</actuator>
 	    </transmission>
-		<transmission name="${prefix}/trans_1">
+		<transmission name="trans_1">
 			<type>transmission_interface/SimpleTransmission</type>
-			<joint name="${prefix}/joint_1"/>
-			<actuator name="${prefix}/motor_1">
+			<joint name="joint_1"/>
+			<actuator name="motor_1">
 				<hardwareInterface>EffortJointInterface</hardwareInterface>
 				<mechanicalReduction>1</mechanicalReduction>
 			</actuator>
 		</transmission>
-		<transmission name="${prefix}/trans_2">
+		<transmission name="trans_2">
 			<type>transmission_interface/SimpleTransmission</type>
-			<joint name="${prefix}/joint_2"/>
-			<actuator name="${prefix}/motor_2">
+			<joint name="joint_2"/>
+			<actuator name="motor_2">
 				<hardwareInterface>EffortJointInterface</hardwareInterface>
 				<mechanicalReduction>1</mechanicalReduction>
 			</actuator>
 		</transmission>
-		<transmission name="${prefix}/trans_3">
+		<transmission name="trans_3">
 			<type>transmission_interface/SimpleTransmission</type>
-			<joint name="${prefix}/joint_3"/>
-			<actuator name="${prefix}/motor_3">
+			<joint name="joint_3"/>
+			<actuator name="motor_3">
 				<hardwareInterface>EffortJointInterface</hardwareInterface>
 				<mechanicalReduction>1</mechanicalReduction>
 			</actuator>
 		</transmission>
-		<transmission name="${prefix}/trans_4">
+		<transmission name="trans_4">
 			<type>transmission_interface/SimpleTransmission</type>
-			<joint name="${prefix}/joint_4"/>
-			<actuator name="${prefix}/motor_4">
+			<joint name="joint_4"/>
+			<actuator name="motor_4">
 				<hardwareInterface>EffortJointInterface</hardwareInterface>
 				<mechanicalReduction>1</mechanicalReduction>
 			</actuator>
 		</transmission>
-		<transmission name="${prefix}/trans_5">
+		<transmission name="trans_5">
 			<type>transmission_interface/SimpleTransmission</type>
-			<joint name="${prefix}/joint_5"/>
-			<actuator name="${prefix}/motor_5">
+			<joint name="joint_5"/>
+			<actuator name="motor_5">
 				<hardwareInterface>EffortJointInterface</hardwareInterface>
 				<mechanicalReduction>1</mechanicalReduction>
 			</actuator>
 		</transmission>
-		<transmission name="${prefix}/trans_6">
+		<transmission name="trans_6">
 			<type>transmission_interface/SimpleTransmission</type>
-			<joint name="${prefix}/joint_6"/>
-			<actuator name="${prefix}/motor_6">
+			<joint name="joint_6"/>
+			<actuator name="motor_6">
 				<hardwareInterface>EffortJointInterface</hardwareInterface>
 				<mechanicalReduction>1</mechanicalReduction>

File: lwr_description/urdf/lwr.urdf.xacro (robot description, xacro)
@@ -14,14 +14,4 @@
    <xacro:property name="d5" value="${damping_factor*1.1}"/>
    <xacro:property name="d6" value="${damping_factor*0.1}"/>
-  <xacro:macro name="gazebo_reference" params="name">
-    <gazebo reference="${name}">
-      <turnGravityOff>
-        false
-      </turnGravityOff>
-      <selfCollide>
-        true
-      </selfCollide>
-    </gazebo>
-  </xacro:macro>
   <!-- Gazebo joint configuration -->
   <xacro:macro  name="gz_joint">
@@ -33,15 +23,15 @@
     <!--<dynamics damping="5.5" friction="1"/>-->
   </xacro:macro>
-   <xacro:macro name="lwr" params="parent name prefix *origin ">
+   <xacro:macro name="lwr" params="parent *origin ">
       <!-- joint between {parent} and lwr_0_link -->
-      <joint name="${prefix}/joint_base" type="fixed">
-        <gazebo reference="${prefix}/joint_base">
+      <joint name="joint_base" type="fixed">
+        <gazebo reference="joint_base">
           <xacro:gz_joint/>
         </gazebo>
          <xacro:insert_block name="origin" />
          <parent link="${parent}" />
-         <child link="${prefix}/link_0" />
-      </joint>
-      <link name="${prefix}/link_0">
+         <child link="link_0" />
+      </joint>
+      <link name="link_0">
           <inertial>
             <origin
@@ -73,10 +63,10 @@
       </link>
       <!-- joint between lwr_0_link and lwr_1_link -->
-      <joint name="${prefix}/joint_0" type="revolute">
-        <gazebo reference="${prefix}/joint_0">
-          <xacro:gz_joint/>
-        </gazebo>
-         <parent link="${prefix}/link_0" />
-         <child link="${prefix}/link_1" />
+      <joint name="joint_0" type="revolute">
+        <gazebo reference="joint_0">
+          <xacro:gz_joint/>
+        </gazebo>
+         <parent link="link_0" />
+         <child link="link_1" />
          <limit lower="${-170 * M_PI / 180}" upper="${170 * M_PI / 180}" effort="${effort_scale * 200}" velocity="${velocity_scale * 112.5 * M_PI / 180}" />
          <dynamics friction="0" damping="${d0}"/>
@@ -84,5 +74,5 @@
          <axis xyz="0 0 1" />
       </joint>
-      <link name="${prefix}/link_1">
+      <link name="link_1">
           <inertial>
             <origin
@@ -114,10 +104,10 @@
       </link>
       <!-- joint between lwr_1_link and lwr_2_link -->
-      <joint name="${prefix}/joint_1" type="revolute">
-        <gazebo reference="${prefix}/joint_1">
-          <xacro:gz_joint/>
-        </gazebo>
-         <parent link="${prefix}/link_1" />
-         <child link="${prefix}/link_2" />
+      <joint name="joint_1" type="revolute">
+        <gazebo reference="joint_1">
+          <xacro:gz_joint/>
+        </gazebo>
+         <parent link="link_1" />
+         <child link="link_2" />
          <limit lower="${-120 * M_PI / 180}" upper="${120 * M_PI / 180}" effort="${effort_scale * 200}" velocity="${velocity_scale * 112.5 * M_PI / 180}" />
          <dynamics friction="0" damping="${d1}"/>
@@ -125,5 +115,5 @@
          <axis xyz="0 -1 0" />
       </joint>
-      <link name="${prefix}/link_2">
+      <link name="link_2">
     <inertial>
       <origin
@@ -163,10 +153,10 @@
       </link>
       <!-- joint between lwr_2_link and lwr_3_link -->
-      <joint name="${prefix}/joint_2" type="revolute">
-        <gazebo reference="${prefix}/joint_2">
-          <xacro:gz_joint/>
-        </gazebo>
-         <parent link="${prefix}/link_2" />
-         <child link="${prefix}/link_3" />
+      <joint name="joint_2" type="revolute">
+        <gazebo reference="joint_2">
+          <xacro:gz_joint/>
+        </gazebo>
+         <parent link="link_2" />
+         <child link="link_3" />
          <limit lower="${-170 * M_PI / 180}" upper="${170 * M_PI / 180}" effort="${effort_scale * 100}" velocity="${velocity_scale * 112.5 * M_PI / 180}" />
          <dynamics friction="0" damping="${d2}"/>
@@ -174,5 +164,5 @@
          <axis xyz="0 0 1" />
       </joint>
-      <link name="${prefix}/link_3">
+      <link name="link_3">
     <inertial>
       <origin
@@ -204,10 +194,10 @@
       </link>
       <!-- joint between lwr_3_link and lwr_4_link -->
-      <joint name="${prefix}/joint_3" type="revolute">
-        <gazebo reference="${prefix}/joint_3">
-          <xacro:gz_joint/>
-        </gazebo>
-         <parent link="${prefix}/link_3" />
-         <child link="${prefix}/link_4" />
+      <joint name="joint_3" type="revolute">
+        <gazebo reference="joint_3">
+          <xacro:gz_joint/>
+        </gazebo>
+         <parent link="link_3" />
+         <child link="link_4" />
          <limit lower="${-120 * M_PI / 180}" upper="${120 * M_PI / 180}" effort="${effort_scale * 100}" velocity="${velocity_scale * 112.5 * M_PI / 180}" />
          <dynamics friction="0" damping="${d3}"/>
@@ -215,5 +205,5 @@
          <axis xyz="0 1 0" />
       </joint>
-      <link name="${prefix}/link_4">
+      <link name="link_4">
     <inertial>
       <origin
@@ -245,10 +235,10 @@
       </link>
       <!-- joint between lwr_4_link and lwr_5_link -->
-      <joint name="${prefix}/joint_4" type="revolute">
-        <gazebo reference="${prefix}/joint_4">
-          <xacro:gz_joint/>
-        </gazebo>
-         <parent link="${prefix}/link_4" />
-         <child link="${prefix}/link_5" />
+      <joint name="joint_4" type="revolute">
+        <gazebo reference="joint_4">
+          <xacro:gz_joint/>
+        </gazebo>
+         <parent link="link_4" />
+         <child link="link_5" />
          <limit lower="${-170 * M_PI / 180}" upper="${170 * M_PI / 180}" effort="${effort_scale * 100}" velocity="${velocity_scale * 180.0 * M_PI / 180}" />
          <dynamics friction="0" damping="${d4}"/>
@@ -256,5 +246,5 @@
          <axis xyz="0 0 1" />
       </joint>
-      <link name="${prefix}/link_5">
+      <link name="link_5">
     <inertial>
       <origin
@@ -286,10 +276,10 @@
       </link>
       <!-- joint between lwr_5_link and lwr_6_link -->
-      <joint name="${prefix}/joint_5" type="revolute">
-        <gazebo reference="${prefix}/joint_5">
-          <xacro:gz_joint/>
-        </gazebo>
-         <parent link="${prefix}/link_5" />
-         <child link="${prefix}/link_6" />
+      <joint name="joint_5" type="revolute">
+        <gazebo reference="joint_5">
+          <xacro:gz_joint/>
+        </gazebo>
+         <parent link="link_5" />
+         <child link="link_6" />
          <limit lower="${-120 * M_PI / 180}" upper="${120 * M_PI / 180}" effort="${effort_scale * 30}" velocity="${velocity_scale * 112.5 * M_PI / 180}" />
          <dynamics friction="0" damping="${d5}"/>
@@ -297,5 +287,5 @@
          <axis xyz="0 -1 0" />
       </joint>
-      <link name="${prefix}/link_6">
+      <link name="link_6">
     <inertial>
       <origin
@@ -327,10 +317,10 @@
       </link>
       <!-- joint between lwr_6_link and lwr_7_link -->
-      <joint name="${prefix}/joint_6" type="revolute">
-        <gazebo reference="${prefix}/joint_6">
-          <xacro:gz_joint/>
-        </gazebo>
-         <parent link="${prefix}/link_6" />
-         <child link="${prefix}/link_7" />
+      <joint name="joint_6" type="revolute">
+        <gazebo reference="joint_6">
+          <xacro:gz_joint/>
+        </gazebo>
+         <parent link="link_6" />
+         <child link="link_7" />
          <limit lower="${-170 * M_PI / 180}" upper="${170 * M_PI / 180}" effort="${effort_scale * 30}" velocity="${velocity_scale * 112.5 * M_PI / 180}" />
          <dynamics friction="0" damping="${d6}"/>
@@ -338,5 +328,5 @@
          <axis xyz="0 0 1" />
       </joint>
-      <link name="${prefix}/link_7">
+      <link name="link_7">
     <inertial>
       <origin

Commit message: add implicit spring damper
Not clear if this affects the gazebo simulation

File: lwr_description/gazebo/lwr.gazebo.urdf.xacro (robot description, xacro)
@@ -1,4 +1,9 @@
 <?xml version="1.0"?>
 <robot xmlns:xacro="http://ros.org/wiki/xacro">
+	<xacro:macro  name="gz_joint" params="joint_name">
+		<gazebo reference="${joint_name}">
+			<implicitSpringDamper>false</implicitSpringDamper>
+		</gazebo>
+	</xacro:macro>
 	<xacro:macro name="lwr_gazebo">
 		<gazebo>
@@ -13,4 +18,11 @@
 			</plugin>
   		</gazebo>
+  		<xacro:gz_joint joint_name="joint_0"/>
+  		<xacro:gz_joint joint_name="joint_1"/>
+  		<xacro:gz_joint joint_name="joint_2"/>
+  		<xacro:gz_joint joint_name="joint_3"/>
+  		<xacro:gz_joint joint_name="joint_4"/>
+  		<xacro:gz_joint joint_name="joint_5"/>
+  		<xacro:gz_joint joint_name="joint_6"/>
 		<gazebo reference="link_0">
 			<gravity>true</gravity>

Commit message: attempt to add ati sensor to gazebo (need gazebo >4.0)

File: lwr_description/gazebo/lwr.gazebo.urdf.xacro (robot description, xacro)
@@ -1,4 +1,5 @@
 <?xml version="1.0"?>
 <robot xmlns:xacro="http://ros.org/wiki/xacro">
+    <xacro:arg name="load_ati_sensor" default="false"/>
 	<xacro:macro  name="gz_joint" params="joint_name">
 		<gazebo reference="${joint_name}">
@@ -9,5 +10,5 @@
 		<gazebo>
 			<plugin name="rtt_gazebo" filename="librtt_gazebo_deployer.so">
-				<robotNamespace>~</robotNamespace>
+				<!--robotNamespace>~</robotNamespace-->
 			  <component>
 			    <package>rtt_lwr_gazebo</package>
@@ -18,4 +19,13 @@
 			</plugin>
   		</gazebo>
+		<!-- ati_sensor NOT YET WORKING (need gazebo >4.0, see ati_sensor.urdf.xacro) -->
+		<!--xacro:if value="$(arg load_ati_sensor)">
+		            <gazebo>
+		                    <plugin name="ati_ft_sensor" filename="libgazebo_ros_ft_sensor.so">
+		                            <jointName>joint_6</jointName>
+		                            <topicName>ft_sensor/FTData</topicName>
+		                    </plugin>
+		            </gazebo>
+		</xacro:if-->
   		<xacro:gz_joint joint_name="joint_0"/>
   		<xacro:gz_joint joint_name="joint_1"/>
@@ -25,7 +35,7 @@
   		<xacro:gz_joint joint_name="joint_5"/>
   		<xacro:gz_joint joint_name="joint_6"/>
-                <gazebo reference="base_link">
-                    <static>true</static>
-                </gazebo>
+        <gazebo reference="base_link">
+            <static>true</static>
+        </gazebo>
 		<gazebo reference="link_0">
 			<gravity>true</gravity>
@@ -58,5 +68,5 @@
 		<gazebo reference="link_7">
 			<gravity>true</gravity>
-			<material>Gazebo/Grey</material>
+			<material>Gazebo/DarkGrey</material>
 		</gazebo>
 	</xacro:macro>

File: lwr_description/urdf/ati_sensor.urdf.xacro (robot description, xacro)
@@ -3,4 +3,6 @@
    <xacro:macro name="ati_sensor">
 	  <joint name="ati_joint" type="fixed">
+	  	<!-- Hack for gazebo <4.0 ati sensor plugin https://bitbucket.org/osrf/gazebo/issues/940/force-torque-sensor-forcetorquesensorcc -->
+	  	<!--limit effort="1000" velocity="0" lower="0" upper="0" /-->
 	    <origin xyz="0 0 0.0488" rpy="0 0 ${(20.0)*M_PI/180.0}" />
 	    <parent link="link_7" />

Commit message: first draft for ati sensor gazebo plugin Need a reset bias option

File: lwr_description/gazebo/lwr.gazebo.urdf.xacro (robot description, xacro)
@@ -19,13 +19,19 @@
 			</plugin>
   		</gazebo>
-		<!-- ati_sensor NOT YET WORKING (need gazebo >4.0, see ati_sensor.urdf.xacro) -->
-		<!--xacro:if value="$(arg load_ati_sensor)">
-		            <gazebo>
-		                    <plugin name="ati_ft_sensor" filename="libgazebo_ros_ft_sensor.so">
-		                            <jointName>joint_6</jointName>
-		                            <topicName>ft_sensor/FTData</topicName>
-		                    </plugin>
-		            </gazebo>
-		</xacro:if-->
+		<!-- ati_sensor (need gazebo >4.0, see ati_sensor.urdf.xacro) -->
+		<xacro:if value="$(arg load_ati_sensor)">
+                    <!-- Use a fixed joint in gazebo -->
+                    <gazebo reference="ati_joint">
+                        <disableFixedJointLumping>true</disableFixedJointLumping>
+                    </gazebo>
+                    <gazebo>
+                        <plugin name="ft_sensor" filename="libgazebo_ros_ft_sensor.so">
+                            <jointName>ati_joint</jointName>
+                            <topicName>ft_sensor/wrench</topicName>
+                            <updateRate>1000</updateRate>
+                            <gaussianNoise>0.0001</gaussianNoise>
+                        </plugin>
+                    </gazebo>
+		</xacro:if>
   		<xacro:gz_joint joint_name="joint_0"/>
   		<xacro:gz_joint joint_name="joint_1"/>
@@ -35,7 +41,7 @@
   		<xacro:gz_joint joint_name="joint_5"/>
   		<xacro:gz_joint joint_name="joint_6"/>
-        <gazebo reference="base_link">
-            <static>true</static>
-        </gazebo>
+                <gazebo reference="base_link">
+                    <static>true</static>
+                </gazebo>
 		<gazebo reference="link_0">
 			<gravity>true</gravity>

File: lwr_description/urdf/ati_sensor.urdf.xacro (robot description, xacro)
@@ -3,6 +3,6 @@
    <xacro:macro name="ati_sensor">
 	  <joint name="ati_joint" type="fixed">
-	  	<!-- Hack for gazebo <4.0 ati sensor plugin https://bitbucket.org/osrf/gazebo/issues/940/force-torque-sensor-forcetorquesensorcc -->
-	  	<!--limit effort="1000" velocity="0" lower="0" upper="0" /-->
+	    <!-- Need the gazebo <disableFixedJointLumping>true</disableFixedJointLumping> option for the gazebo ros pkgs ft_sensor -->
+	    <limit effort="400" velocity="0" lower="0" upper="0" />
 	    <origin xyz="0 0 0.0488" rpy="0 0 ${(20.0)*M_PI/180.0}" />
 	    <parent link="link_7" />
