Commit message: ati ft is now the real sensing surface of the sensor

File: lwr_description/gazebo/lwr.gazebo.urdf.xacro (robot description, xacro)
@@ -4,4 +4,5 @@
 	<xacro:macro  name="gz_joint" params="joint_name">
 		<gazebo reference="${joint_name}">
+			<provideFeedback>true</provideFeedback>
 			<implicitSpringDamper>true</implicitSpringDamper>
 		</gazebo>
@@ -22,5 +23,9 @@
 		<xacro:if value="$(arg load_ati_sensor)">
                     <!-- Use a fixed joint in gazebo -->
+                    <gazebo reference="ati_base_joint">
+                        <disableFixedJointLumping>true</disableFixedJointLumping>
+                    </gazebo>
                     <gazebo reference="ati_joint">
+			<provideFeedback>true</provideFeedback>
                         <disableFixedJointLumping>true</disableFixedJointLumping>
                     </gazebo>

File: lwr_description/urdf/ati_sensor.urdf.xacro (robot description, xacro)
@@ -2,32 +2,32 @@
 <robot xmlns:xacro="http://www.ros.org/wiki/xacro">
    <xacro:macro name="ati_sensor">
-	  <joint name="ati_joint" type="fixed">
+	  <joint name="ati_base_joint" type="fixed">
 	    <!-- Need the gazebo <disableFixedJointLumping>true</disableFixedJointLumping> option for the gazebo ros pkgs ft_sensor -->
 	    <limit effort="400" velocity="0" lower="0" upper="0" />
-	    <origin xyz="0 0 0.0488" rpy="0 0 ${(20.0)*M_PI/180.0}" />
+	    <origin xyz="0 0 0.045" rpy="0 0 ${(20.0)*M_PI/180.0}" />
 	    <parent link="link_7" />
-	    <child link="ati_link" />
+	    <child link="ati_base_link" />
 	  </joint>
-	  <link name="ati_link">
-	    <inertial>
-	      <origin
-		xyz="-0.00178553387370124 -0.000310330841277809 0.0197116137003042"
-		rpy="0 0 0" />
-	      <mass
-		value="0.316951020394394" />
-	      <inertia
-		ixx="0.000196894344101305"
-		ixy="4.02893385807679E-06"
-		ixz="-6.2186338186242E-06"
-		iyy="0.000219267703175818"
-		iyz="-1.08082570436843E-06"
-		izz="0.000295322983266294" />
-	    </inertial>
+	  <link name="ati_base_link">
+		  <inertial>
+		    <origin
+		      xyz="-0.00480740431783837 0.00412111608218374 -0.0111556038816137"
+		      rpy="0 0 0" />
+		    <mass
+		      value="0.316951020394394" />
+		    <inertia
+		      ixx="4.36061005979496E-05"
+		      ixy="-1.11387576114314E-05"
+		      ixz="1.18766045084891E-06"
+		      iyy="4.67870488895371E-05"
+		      iyz="-1.05981886988621E-06"
+		      izz="7.64371245181666E-05" />
+		  </inertial>
 	    <visual>
-	      <origin xyz="0 0 -0.0488" rpy="0 0 ${-45*M_PI/180.0}" />
+	      <origin xyz="0 0 0.0" rpy="0 0 0" />
 	      <geometry>
 		<mesh filename="package://lwr_description/meshes/ati_sensor/ati_sensor.stl" />
 	      </geometry>
-      	      <material name="color_j7"/>
+				<material name="color_j7"/>
 	    </visual>
 	    <collision>
@@ -38,4 +38,49 @@
 	    </collision>
 	  </link>
+  <joint name="ati_joint" type="fixed">
+    <limit effort="400" velocity="0" lower="0" upper="0" />
+    <origin xyz="0 0 0.0036" rpy="0 0 0" />
+    <parent link="ati_base_link" />
+    <child link="ati_link" />
+  </joint>
+  <link name="ati_link">
+    <inertial>
+      <origin
+        xyz="-1.59594559789866E-16 -6.93889390390723E-17 -0.00209999999999987"
+        rpy="0 0 0" />
+      <mass
+        value="0.001" />
+      <inertia
+        ixx="2.04554394204082E-06"
+        ixy="-2.11758236813575E-22"
+        ixz="-1.11092775809582E-23"
+        iyy="2.04554394204082E-06"
+        iyz="-8.96327424295973E-24"
+        izz="4.07793678453489E-06" />
+    </inertial>
+    <visual>
+      <origin
+        xyz="0 0 0"
+        rpy="0 0 0" />
+      <geometry>
+        <mesh
+          filename="package://lwr_description/meshes/ati_sensor/ati_sensor_cylinder.stl" />
+      </geometry>
+      <material
+        name="">
+        <color
+          rgba="0.792156862745098 0.819607843137255 0.933333333333333 1" />
+      </material>
+    </visual>
+    <collision>
+      <origin
+        xyz="0 0 0"
+        rpy="0 0 0" />
+      <geometry>
+        <mesh
+          filename="package://lwr_description/meshes/ati_sensor/ati_sensor_cylinder.stl" />
+      </geometry>
+    </collision>
+  </link>
    </xacro:macro>
 </robot>

Commit message: add some extra color info Problem is that fixed links are merge in color

File: lwr_description/gazebo/lwr.gazebo.urdf.xacro (robot description, xacro)
@@ -2,4 +2,7 @@
 <robot xmlns:xacro="http://ros.org/wiki/xacro">
     <xacro:arg name="load_ati_sensor" default="false"/>
+    <xacro:arg name="load_base" default="false"/>
+    <xacro:arg name="load_handle" default="false"/>
+    <xacro:arg name="load_calib_tool" default="false"/>
 	<xacro:macro  name="gz_joint" params="joint_name">
 		<gazebo reference="${joint_name}">
@@ -30,4 +33,10 @@
                         <disableFixedJointLumping>true</disableFixedJointLumping>
                     </gazebo>
+                    <gazebo reference="ati_base_link">
+                        <material>Gazebo/Grey</material>
+                    </gazebo>
+                    <gazebo reference="ati_link">
+                        <material>Gazebo/Grey</material>
+                    </gazebo>
                     <gazebo>
                         <plugin name="ft_sensor" filename="libgazebo_ros_ft_sensor.so">
@@ -39,4 +48,25 @@
                     </gazebo>
 		</xacro:if>
+                <xacro:if value="$(arg load_handle)">
+                    <gazebo reference="handle_link">
+                        <material>Gazebo/White</material>
+                    </gazebo>
+                </xacro:if>
+                <xacro:if value="$(arg load_base)">
+                    <gazebo reference="base_link">
+                        <material>Gazebo/Grey</material>
+                    </gazebo>
+                </xacro:if>
+                <!-- base_link and link_0 are fixed, so merged by gazebo -->
+                <xacro:unless value="$(arg load_base)">
+                    <gazebo reference="base_link">
+                        <material>Gazebo/Orange</material>
+                    </gazebo>
+                </xacro:unless>
+                <xacro:if value="$(arg load_calib_tool)">
+                    <gazebo reference="calib_link">
+                        <material>Gazebo/White</material>
+                    </gazebo>
+                </xacro:if>
   		<xacro:gz_joint joint_name="joint_0"/>
   		<xacro:gz_joint joint_name="joint_1"/>
@@ -46,37 +76,23 @@
   		<xacro:gz_joint joint_name="joint_5"/>
   		<xacro:gz_joint joint_name="joint_6"/>
-                <gazebo reference="base_link">
-                    <static>true</static>
-                </gazebo>
-		<gazebo reference="link_0">
-			<gravity>true</gravity>
-			<material>Gazebo/Orange</material>
-		</gazebo>
 		<gazebo reference="link_1">
-			<gravity>true</gravity>
 			<material>Gazebo/Orange</material>
 		</gazebo>
 		<gazebo reference="link_2">
-			<gravity>true</gravity>
 			<material>Gazebo/Orange</material>
 		</gazebo>
 		<gazebo reference="link_3">
-			<gravity>true</gravity>
 			<material>Gazebo/Orange</material>
 		</gazebo>
 		<gazebo reference="link_4">
-			<gravity>true</gravity>
 			<material>Gazebo/Orange</material>
 		</gazebo>
 		<gazebo reference="link_5">
-			<gravity>true</gravity>
 			<material>Gazebo/Orange</material>
 		</gazebo>
 		<gazebo reference="link_6">
-			<gravity>true</gravity>
 			<material>Gazebo/Grey</material>
 		</gazebo>
 		<gazebo reference="link_7">
-			<gravity>true</gravity>
 			<material>Gazebo/DarkGrey</material>
 		</gazebo>

Commit message: add gz state pub (test)

File: lwr_description/gazebo/lwr.gazebo.urdf.xacro (robot description, xacro)
@@ -5,4 +5,14 @@
     <xacro:arg name="load_handle" default="false"/>
     <xacro:arg name="load_calib_tool" default="false"/>
+    <xacro:macro name="gz_ft_sensor" params="joint_name">
+        <gazebo>
+            <plugin name="ft_sensor_${joint_name}" filename="libgazebo_ros_ft_sensor.so">
+                <jointName>${joint_name}</jointName>
+                <topicName>lwr_gazebo/ft_sensor_${joint_name}</topicName>
+                <updateRate>1000</updateRate>
+                <gaussianNoise>0.0001</gaussianNoise>
+            </plugin>
+        </gazebo>
+     </xacro:macro>
 	<xacro:macro  name="gz_joint" params="joint_name">
 		<gazebo reference="${joint_name}">
@@ -55,4 +65,12 @@
                     </gazebo>
 		</xacro:if>
+            <gazebo>
+    			<plugin name="gz_state_pub" filename="libgazebo_ros_joint_state_publisher.so">
+    				<!--robotNamespace>~</robotNamespace-->
+                  <jointName>joint_0,joint_1,joint_2,joint_3,joint_4,joint_5,joint_6</jointName>
+    			  <updateRate>100</updateRate>
+                  <alwaysOn>true</alwaysOn>
+    			</plugin>
+            </gazebo>
                 <xacro:if value="$(arg load_handle)">
                     <gazebo reference="handle_link">
@@ -83,4 +101,11 @@
   		<xacro:gz_joint joint_name="joint_5"/>
   		<xacro:gz_joint joint_name="joint_6"/>
+        <!--xacro:gz_ft_sensor joint_name="joint_0"/-->
+        <!--xacro:gz_ft_sensor joint_name="joint_1"/-->
+        <!--xacro:gz_ft_sensor joint_name="joint_2"/-->
+        <!--xacro:gz_ft_sensor joint_name="joint_3"/-->
+        <!--xacro:gz_ft_sensor joint_name="joint_4"/-->
+        <!--xacro:gz_ft_sensor joint_name="joint_5"/-->
+        <!--xacro:gz_ft_sensor joint_name="joint_6"/-->
 		<gazebo reference="link_1">
 			<material>Gazebo/Orange</material>

Commit message: Adding the load_gripper argument

File: lwr_description/gazebo/lwr.gazebo.urdf.xacro (robot description, xacro)
@@ -4,4 +4,5 @@
     <xacro:arg name="load_base" default="false"/>
     <xacro:arg name="load_handle" default="false"/>
+    <xacro:arg name="load_gripper" default="false"/>
     <xacro:arg name="load_calib_tool" default="false"/>
 	<xacro:macro  name="gz_joint" params="joint_name">
@@ -60,4 +61,9 @@
                     </gazebo>
                 </xacro:if>
+                <xacro:if value="$(arg load_handle)">
+                    <gazebo reference="gripper_base_link">
+                        <material>Gazebo/White</material>
+                    </gazebo>
+                </xacro:if>
                 <xacro:if value="$(arg load_base)">
                     <gazebo reference="base_link">

Commit message: reindent file

File: lwr_description/gazebo/lwr.gazebo.urdf.xacro (robot description, xacro)
@@ -16,108 +16,110 @@
             </plugin>
         </gazebo>
-     </xacro:macro>
-	<xacro:macro  name="gz_joint" params="joint_name">
-		<gazebo reference="${joint_name}">
-			<provideFeedback>true</provideFeedback>
+    </xacro:macro>
+    <xacro:macro  name="gz_joint" params="joint_name">
+        <gazebo reference="${joint_name}">
+            <provideFeedback>true</provideFeedback>
             <!-- Dangerous option :) -->
-			<!--implicitSpringDamper>true</implicitSpringDamper-->
-                        <!--stopCfm>0.9</stopCfm-->
-                        <!--stopErp>0.5</stopErp-->
-		</gazebo>
-	</xacro:macro>
-	<xacro:macro name="lwr_gazebo">
-		<!-- ati_sensor (need gazebo >4.0, see ati_sensor.urdf.xacro) -->
-		<xacro:if value="$(arg load_ati_sensor)">
-                    <!-- Use a fixed joint in gazebo -->
-                    <gazebo reference="ati_base_joint">
-                        <disableFixedJointLumping>true</disableFixedJointLumping>
-                    </gazebo>
-                    <gazebo reference="ati_joint">
-			<provideFeedback>true</provideFeedback>
-                        <disableFixedJointLumping>true</disableFixedJointLumping>
-                    </gazebo>
-                    <gazebo reference="ati_base_link">
-                        <material>Gazebo/Grey</material>
-                    </gazebo>
-                    <gazebo reference="ati_link">
-                        <!-- gravity tag does not work for some reason ,
-                        so we have to update the lwr_gazebo ops
-                        with lwr_gazebo.setLinkGravityMode("ati_link",false) -->
-                        <gravity>false</gravity>
-                        <material>Gazebo/Grey</material>
-                    </gazebo>
-                    <gazebo>
-                        <plugin name="ft_sensor" filename="libgazebo_ros_ft_sensor.so">
-                            <robotNamespace>ft_sensor</robotNamespace>
-                            <jointName>ati_joint</jointName>
-                            <topicName>wrench</topicName>
-                            <updateRate>1000</updateRate>
-                            <gaussianNoise>0.0001</gaussianNoise>
-                        </plugin>
-                    </gazebo>
-		</xacro:if>
-            <!--gazebo>
-    			<plugin name="gz_state_pub" filename="libgazebo_ros_joint_state_publisher.so">
-                  <jointName>joint_0,joint_1,joint_2,joint_3,joint_4,joint_5,joint_6</jointName>
-    			  <updateRate>100</updateRate>
-                  <alwaysOn>true</alwaysOn>
-    			</plugin>
-            </gazebo-->
-                <xacro:if value="$(arg load_handle)">
-                    <gazebo reference="handle_link">
-                        <material>Gazebo/White</material>
-                    </gazebo>
-                </xacro:if>
-                <xacro:if value="$(arg load_base)">
-                    <gazebo reference="base_link">
-                        <material>Gazebo/Grey</material>
-                    </gazebo>
-                </xacro:if>
-                <!-- base_link and link_0 are fixed, so merged by gazebo -->
-                <xacro:unless value="$(arg load_base)">
-                    <gazebo reference="base_link">
-                        <material>Gazebo/Orange</material>
-                    </gazebo>
-                </xacro:unless>
-                <xacro:if value="$(arg load_calib_tool)">
-                    <gazebo reference="calib_link">
-                        <material>Gazebo/White</material>
-                    </gazebo>
-                </xacro:if>
-  		<xacro:gz_joint joint_name="joint_0"/>
-  		<xacro:gz_joint joint_name="joint_1"/>
-  		<xacro:gz_joint joint_name="joint_2"/>
-  		<xacro:gz_joint joint_name="joint_3"/>
-  		<xacro:gz_joint joint_name="joint_4"/>
-  		<xacro:gz_joint joint_name="joint_5"/>
-  		<xacro:gz_joint joint_name="joint_6"/>
-        <!--xacro:gz_ft_sensor joint_name="joint_0"/-->
-        <!--xacro:gz_ft_sensor joint_name="joint_1"/-->
-        <!--xacro:gz_ft_sensor joint_name="joint_2"/-->
-        <!--xacro:gz_ft_sensor joint_name="joint_3"/-->
-        <!--xacro:gz_ft_sensor joint_name="joint_4"/-->
-        <!--xacro:gz_ft_sensor joint_name="joint_5"/-->
-        <!--xacro:gz_ft_sensor joint_name="joint_6"/-->
-		<gazebo reference="link_1">
-			<material>Gazebo/Orange</material>
-		</gazebo>
-		<gazebo reference="link_2">
-			<material>Gazebo/Orange</material>
-		</gazebo>
-		<gazebo reference="link_3">
-			<material>Gazebo/Orange</material>
-		</gazebo>
-		<gazebo reference="link_4">
-			<material>Gazebo/Orange</material>
-		</gazebo>
-		<gazebo reference="link_5">
-			<material>Gazebo/Orange</material>
-		</gazebo>
-		<gazebo reference="link_6">
-			<material>Gazebo/Grey</material>
-		</gazebo>
-		<gazebo reference="link_7">
-			<material>Gazebo/DarkGrey</material>
-		</gazebo>
-	</xacro:macro>
+            <!--implicitSpringDamper>true</implicitSpringDamper-->
+            <!--stopCfm>0.9</stopCfm-->
+            <!--stopErp>0.5</stopErp-->
+        </gazebo>
+    </xacro:macro>
+    <xacro:macro name="lwr_gazebo">
+        <!-- ati_sensor (need gazebo >4.0, see ati_sensor.urdf.xacro) -->
+        <xacro:if value="$(arg load_ati_sensor)">
+            <!-- Use a fixed joint in gazebo -->
+            <gazebo reference="ati_base_joint">
+                <disableFixedJointLumping>true</disableFixedJointLumping>
+            </gazebo>
+            <gazebo reference="ati_joint">
+                <provideFeedback>true</provideFeedback>
+                <disableFixedJointLumping>true</disableFixedJointLumping>
+            </gazebo>
+            <gazebo reference="ati_base_link">
+                <material>Gazebo/Grey</material>
+            </gazebo>
+            <gazebo reference="ati_link">
+                <!-- gravity tag does not work for some reason ,
+                so we have to update the lwr_gazebo ops
+                with lwr_gazebo.setLinkGravityMode("ati_link",false) -->
+                <gravity>false</gravity>
+                <material>Gazebo/Grey</material>
+            </gazebo>
+            <gazebo>
+                <plugin name="ft_sensor" filename="libgazebo_ros_ft_sensor.so">
+                    <robotNamespace>ft_sensor</robotNamespace>
+                    <jointName>ati_joint</jointName>
+                    <topicName>wrench</topicName>
+                    <updateRate>1000</updateRate>
+                    <gaussianNoise>0.0001</gaussianNoise>
+                </plugin>
+            </gazebo>
+        </xacro:if>
+        <!-- The state publisher is done by the RTTStatePublisher() as on the real HW -->
+        <!--gazebo>
+        <plugin name="gz_state_pub" filename="libgazebo_ros_joint_state_publisher.so">
+        <jointName>joint_0,joint_1,joint_2,joint_3,joint_4,joint_5,joint_6</jointName>
+        <updateRate>100</updateRate>
+        <alwaysOn>true</alwaysOn>
+    </plugin>
+</gazebo-->
+<xacro:if value="$(arg load_handle)">
+    <gazebo reference="handle_link">
+        <material>Gazebo/White</material>
+    </gazebo>
+</xacro:if>
+<xacro:if value="$(arg load_base)">
+    <gazebo reference="base_link">
+        <material>Gazebo/Grey</material>
+    </gazebo>
+</xacro:if>
+<!-- base_link and link_0 are fixed, so merged by gazebo -->
+<xacro:unless value="$(arg load_base)">
+    <gazebo reference="base_link">
+        <material>Gazebo/Orange</material>
+    </gazebo>
+</xacro:unless>
+<xacro:if value="$(arg load_calib_tool)">
+    <gazebo reference="calib_link">
+        <material>Gazebo/White</material>
+    </gazebo>
+</xacro:if>
+<xacro:gz_joint joint_name="joint_0"/>
+<xacro:gz_joint joint_name="joint_1"/>
+<xacro:gz_joint joint_name="joint_2"/>
+<xacro:gz_joint joint_name="joint_3"/>
+<xacro:gz_joint joint_name="joint_4"/>
+<xacro:gz_joint joint_name="joint_5"/>
+<xacro:gz_joint joint_name="joint_6"/>
+<!-- If you want to add a Joint Torque sensor at each Joint -->
+<!--xacro:gz_ft_sensor joint_name="joint_0"/-->
+<!--xacro:gz_ft_sensor joint_name="joint_1"/-->
+<!--xacro:gz_ft_sensor joint_name="joint_2"/-->
+<!--xacro:gz_ft_sensor joint_name="joint_3"/-->
+<!--xacro:gz_ft_sensor joint_name="joint_4"/-->
+<!--xacro:gz_ft_sensor joint_name="joint_5"/-->
+<!--xacro:gz_ft_sensor joint_name="joint_6"/-->
+<gazebo reference="link_1">
+    <material>Gazebo/Orange</material>
+</gazebo>
+<gazebo reference="link_2">
+    <material>Gazebo/Orange</material>
+</gazebo>
+<gazebo reference="link_3">
+    <material>Gazebo/Orange</material>
+</gazebo>
+<gazebo reference="link_4">
+    <material>Gazebo/Orange</material>
+</gazebo>
+<gazebo reference="link_5">
+    <material>Gazebo/Orange</material>
+</gazebo>
+<gazebo reference="link_6">
+    <material>Gazebo/Grey</material>
+</gazebo>
+<gazebo reference="link_7">
+    <material>Gazebo/DarkGrey</material>
+</gazebo>
+</xacro:macro>
 </robot>

Commit message: fix misplaced args

File: lwr_description/gazebo/lwr.gazebo.urdf.xacro (robot description, xacro)
@@ -56,4 +56,14 @@
                 </plugin>
             </gazebo>
+            <xacro:if value="$(arg load_handle)">
+                <gazebo reference="handle_link">
+                    <material>Gazebo/White</material>
+                </gazebo>
+            </xacro:if>
+            <xacro:if value="$(arg load_calib_tool)">
+                <gazebo reference="calib_link">
+                    <material>Gazebo/White</material>
+                </gazebo>
+            </xacro:if>
         </xacro:if>
         <!-- The state publisher is done by the RTTStatePublisher() as on the real HW -->
@@ -65,9 +75,4 @@
     </plugin>
 </gazebo-->
-<xacro:if value="$(arg load_handle)">
-    <gazebo reference="handle_link">
-        <material>Gazebo/White</material>
-    </gazebo>
-</xacro:if>
 <xacro:if value="$(arg load_base)">
     <gazebo reference="base_link">
@@ -81,9 +86,4 @@
     </gazebo>
 </xacro:unless>
-<xacro:if value="$(arg load_calib_tool)">
-    <gazebo reference="calib_link">
-        <material>Gazebo/White</material>
-    </gazebo>
-</xacro:if>
 <xacro:gz_joint joint_name="joint_0"/>
 <xacro:gz_joint joint_name="joint_1"/>

Commit message: Update camera config for gazebo

File: lwr_description/gazebo/lwr.gazebo.urdf.xacro (robot description, xacro)
@@ -48,5 +48,5 @@
                 <material>Gazebo/Grey</material>
             </gazebo>
-            <gazebo reference="cam_link">
+            <gazebo reference="head_cam_link">
               <sensor name="head_cam" type="camera">
                 <update_rate>30</update_rate>
@@ -69,5 +69,5 @@
                   <imageTopicName>image_raw</imageTopicName>
                   <cameraInfoTopicName>camera_info</cameraInfoTopicName>
-                  <frameName>cam_link_optical</frameName>
+                  <frameName>head_cam_link_optical</frameName>
                   <hackBaseline>0.07</hackBaseline>
                   <distortionK1>-0.424180</distortionK1>

File: lwr_description/urdf/head_cam.urdf.xacro (robot description, xacro)
@@ -38,4 +38,13 @@
         <axis xyz="0 0 0" />
     </joint>
+    <link name="head_cam_link_optical" />
+    <joint name="head_cam_optical_joint" type="fixed">
+      <!-- these values have to be these values otherwise the gazebo camera
+          image won't be aligned properly with the frame it is supposedly
+          originating from -->
+      <origin xyz="0 0 0" rpy="-1.570796 0 -1.570796"/>
+      <parent link="head_cam_link"/>
+      <child link="head_cam_link_optical"/>
+    </joint>
   </xacro:macro>
 </robot>
