Commit message: enable self collision

File: lwr_description/gazebo/lwr.gazebo.urdf.xacro (robot description, xacro)
@@ -7,4 +7,5 @@
     <xacro:arg name="load_hook" default="false"/>
     <xacro:arg name="load_gazebo_ros_control" default="false"/>
+    <xacro:arg name="load_model_joint_plugin" default="false"/>
     <xacro:arg name="robot_name" default="lwr"/>
     <xacro:macro name="gz_ft_sensor" params="joint_name">
@@ -25,4 +26,9 @@
             <!--stopCfm>0.9</stopCfm-->
             <!--stopErp>0.5</stopErp-->
+        </gazebo>
+    </xacro:macro>
+    <xacro:macro  name="enable_self_collision" params="link_name">
+        <gazebo reference="${link_name}">
+            <self_collide>true</self_collide>
         </gazebo>
     </xacro:macro>
@@ -107,11 +113,13 @@
             </xacro:if>
         </xacro:if>
-        <gazebo>
-            <plugin name="model_joint_plugin" filename="libmodel_joint_plugin.so">
-                <!-- <robotNamespace>~</robotNamespace> -->
-                <topicName>~/$(arg robot_name)/joint_states</topicName>
-                <numberOfStepsBeforeSync>10</numberOfStepsBeforeSync>
-            </plugin>
-        </gazebo>
+        <xacro:if value="$(arg load_model_joint_plugin)">
+            <gazebo>
+                <plugin name="model_joint_plugin" filename="libmodel_joint_plugin.so">
+                    <!-- <robotNamespace>~</robotNamespace> -->
+                    <topicName>~/$(arg robot_name)/joint_states</topicName>
+                    <numberOfStepsBeforeSync>10</numberOfStepsBeforeSync>
+                </plugin>
+            </gazebo>
+        </xacro:if>
         <!-- The state publisher is done by the RTTStatePublisher() as on the real HW -->
         <!--gazebo>
@@ -140,4 +148,19 @@
 <xacro:gz_joint joint_name="joint_5"/>
 <xacro:gz_joint joint_name="joint_6"/>
+<xacro:enable_self_collision link_name="table_link"/>
+<xacro:enable_self_collision link_name="screwdriver_link"/>
+<!-- <xacro:enable_self_collision link_name="ati_link"/> -->
+<xacro:enable_self_collision link_name="base_link"/>
+<xacro:enable_self_collision link_name="link_0"/>
+<xacro:enable_self_collision link_name="link_1"/>
+<xacro:enable_self_collision link_name="link_2"/>
+<xacro:enable_self_collision link_name="link_3"/>
+<xacro:enable_self_collision link_name="link_4"/>
+<xacro:enable_self_collision link_name="link_5"/>
+<xacro:enable_self_collision link_name="link_6"/>
+<xacro:enable_self_collision link_name="link_7"/>
+<xacro:enable_self_collision link_name="hook_link"/>
+<xacro:enable_self_collision link_name="head_cam_link"/>
+<xacro:enable_self_collision link_name="handle_link"/>
 <!-- If you want to add a Joint Torque sensor at each Joint -->
 <!--xacro:gz_ft_sensor joint_name="joint_0"/-->

Commit message: Update description for rtt_lwr-1.0

File: lwr_description/gazebo/lwr.gazebo.urdf.xacro (robot description, xacro)
@@ -1,107 +1,186 @@
 <?xml version="1.0"?>
 <robot xmlns:xacro="http://ros.org/wiki/xacro">
+    <xacro:arg name="load_base" default="false"/>
     <xacro:arg name="load_ati_sensor" default="false"/>
-    <xacro:arg name="load_base" default="false"/>
+    <xacro:arg name="load_calib_tool" default="false"/>
     <xacro:arg name="load_handle" default="false"/>
-    <xacro:arg name="load_calib_tool" default="false"/>
-	<xacro:macro  name="gz_joint" params="joint_name">
-		<gazebo reference="${joint_name}">
-			<provideFeedback>true</provideFeedback>
+    <xacro:arg name="load_hook" default="false"/>
+    <xacro:arg name="load_gazebo_ros_control" default="false"/>
+    <xacro:arg name="load_model_joint_plugin" default="false"/>
+    <xacro:arg name="robot_name" default="lwr"/>
+    <xacro:macro name="gz_ft_sensor" params="joint_name">
+        <gazebo>
+            <plugin name="ft_sensor_${joint_name}" filename="libgazebo_ros_ft_sensor.so">
+                <jointName>${joint_name}</jointName>
+                <topicName>~/ft_sensor_${joint_name}</topicName>
+                <updateRate>1000</updateRate>
+                <gaussianNoise>0.0001</gaussianNoise>
+            </plugin>
+        </gazebo>
+    </xacro:macro>
+    <xacro:macro  name="gz_joint" params="joint_name">
+        <gazebo reference="${joint_name}">
+            <provideFeedback>true</provideFeedback>
             <!-- Dangerous option :) -->
-			<!--implicitSpringDamper>true</implicitSpringDamper-->
-                        <!--stopCfm>0.9</stopCfm-->
-                        <!--stopErp>0.5</stopErp-->
-		</gazebo>
-	</xacro:macro>
-	<xacro:macro name="lwr_gazebo">
-		<gazebo>
-			<plugin name="rtt_gazebo" filename="librtt_gazebo_deployer.so">
-				<!--robotNamespace>~</robotNamespace-->
-			  <component>
-			    <package>rtt_lwr_gazebo</package>
-			    <type>LWRGazeboComponent</type>
-			    <name>lwr_gazebo</name>
-			  </component>
-			    <orocosScript><filename>$(find rtt_lwr_gazebo)/scripts/lwr_gazebo.ops</filename></orocosScript>
-			</plugin>
-  		</gazebo>
-		<!-- ati_sensor (need gazebo >4.0, see ati_sensor.urdf.xacro) -->
-		<xacro:if value="$(arg load_ati_sensor)">
-                    <!-- Use a fixed joint in gazebo -->
-                    <gazebo reference="ati_base_joint">
-                        <disableFixedJointLumping>true</disableFixedJointLumping>
-                    </gazebo>
-                    <gazebo reference="ati_joint">
-			<provideFeedback>true</provideFeedback>
-                        <disableFixedJointLumping>true</disableFixedJointLumping>
-                    </gazebo>
-                    <gazebo reference="ati_base_link">
-                        <material>Gazebo/Grey</material>
-                    </gazebo>
-                    <gazebo reference="ati_link">
-                        <!-- gravity tag does not work for some reason ,
-                        so we have to update the lwr_gazebo ops
-                        with lwr_gazebo.setLinkGravityMode("ati_link",false) -->
-                        <gravity>false</gravity>
-                        <material>Gazebo/Grey</material>
-                    </gazebo>
-                    <gazebo>
-                        <plugin name="ft_sensor" filename="libgazebo_ros_ft_sensor.so">
-                            <jointName>ati_joint</jointName>
-                            <topicName>ft_sensor/wrench</topicName>
-                            <updateRate>1000</updateRate>
-                            <gaussianNoise>0.0001</gaussianNoise>
-                        </plugin>
-                    </gazebo>
-		</xacro:if>
-                <xacro:if value="$(arg load_handle)">
-                    <gazebo reference="handle_link">
-                        <material>Gazebo/White</material>
-                    </gazebo>
-                </xacro:if>
-                <xacro:if value="$(arg load_base)">
-                    <gazebo reference="base_link">
-                        <material>Gazebo/Grey</material>
-                    </gazebo>
-                </xacro:if>
-                <!-- base_link and link_0 are fixed, so merged by gazebo -->
-                <xacro:unless value="$(arg load_base)">
-                    <gazebo reference="base_link">
-                        <material>Gazebo/Orange</material>
-                    </gazebo>
-                </xacro:unless>
-                <xacro:if value="$(arg load_calib_tool)">
-                    <gazebo reference="calib_link">
-                        <material>Gazebo/White</material>
-                    </gazebo>
-                </xacro:if>
-  		<xacro:gz_joint joint_name="joint_0"/>
-  		<xacro:gz_joint joint_name="joint_1"/>
-  		<xacro:gz_joint joint_name="joint_2"/>
-  		<xacro:gz_joint joint_name="joint_3"/>
-  		<xacro:gz_joint joint_name="joint_4"/>
-  		<xacro:gz_joint joint_name="joint_5"/>
-  		<xacro:gz_joint joint_name="joint_6"/>
-		<gazebo reference="link_1">
-			<material>Gazebo/Orange</material>
-		</gazebo>
-		<gazebo reference="link_2">
-			<material>Gazebo/Orange</material>
-		</gazebo>
-		<gazebo reference="link_3">
-			<material>Gazebo/Orange</material>
-		</gazebo>
-		<gazebo reference="link_4">
-			<material>Gazebo/Orange</material>
-		</gazebo>
-		<gazebo reference="link_5">
-			<material>Gazebo/Orange</material>
-		</gazebo>
-		<gazebo reference="link_6">
-			<material>Gazebo/Grey</material>
-		</gazebo>
-		<gazebo reference="link_7">
-			<material>Gazebo/DarkGrey</material>
-		</gazebo>
-	</xacro:macro>
+            <!--implicitSpringDamper>true</implicitSpringDamper-->
+            <!--stopCfm>0.9</stopCfm-->
+            <!--stopErp>0.5</stopErp-->
+        </gazebo>
+    </xacro:macro>
+    <xacro:macro  name="enable_self_collision" params="link_name">
+        <gazebo reference="${link_name}">
+            <self_collide>true</self_collide>
+        </gazebo>
+    </xacro:macro>
+    <xacro:macro name="lwr_gazebo">
+        <xacro:if value="$(arg load_gazebo_ros_control)">
+            <gazebo>
+              <plugin name="gazebo_ros_control" filename="libgazebo_ros_control.so">
+                <!-- <robotNamespace>/</robotNamespace> -->
+              </plugin>
+            </gazebo>
+        </xacro:if>
+        <!-- ati_sensor (need gazebo >4.0, see ati_sensor.urdf.xacro) -->
+        <xacro:if value="$(arg load_ati_sensor)">
+            <!-- Use a fixed joint in gazebo -->
+            <gazebo reference="ati_base_joint">
+                <disableFixedJointLumping>true</disableFixedJointLumping>
+            </gazebo>
+            <gazebo reference="ati_joint">
+                <provideFeedback>true</provideFeedback>
+                <disableFixedJointLumping>true</disableFixedJointLumping>
+            </gazebo>
+            <gazebo reference="ati_base_link">
+                <material>Gazebo/Grey</material>
+            </gazebo>
+            <gazebo reference="head_cam_link">
+              <sensor name="head_cam" type="camera">
+                <update_rate>30</update_rate>
+                <camera name="head_cam">
+                  <horizontal_fov>0.6126</horizontal_fov>
+                  <image>
+                    <width>1360</width>
+                    <height>1024</height>
+                    <format>R8G8B8</format>
+                  </image>
+                  <clip>
+                    <near>0.02</near>
+                    <far>300</far>
+                  </clip>
+                </camera>
+                <plugin name='camera_controller' filename='libgazebo_ros_camera.so'>
+                  <alwaysOn>true</alwaysOn>
+                  <updateRate>30.0</updateRate>
+                  <cameraName>head_cam</cameraName>
+                  <imageTopicName>image_raw</imageTopicName>
+                  <cameraInfoTopicName>camera_info</cameraInfoTopicName>
+                  <frameName>head_cam_link_optical</frameName>
+                  <hackBaseline>0.07</hackBaseline>
+                  <!--distortionK1>-0.424180</distortionK1-->
+                  <!--distortionK2>0.622783</distortionK2-->
+                  <!--distortionK3>-0.004707</distortionK3-->
+                  <!--distortionT1>-0.000359</distortionT1-->
+                  <!--distortionT2>0.0</distortionT2-->
+                  <CxPrime>0</CxPrime>
+                  <Cx>0</Cx>
+                  <Cy>0</Cy>
+                  <focalLength>2150.179542</focalLength>
+                  </plugin>
+                </sensor>
+              </gazebo>
+            <gazebo reference="ati_link">
+                <gravity>false</gravity>
+                <material>Gazebo/Grey</material>
+            </gazebo>
+            <gazebo>
+                <plugin name="ft_sensor" filename="libgazebo_ros_ft_sensor.so">
+                    <robotNamespace>ft_sensor</robotNamespace>
+                    <jointName>ati_joint</jointName>
+                    <topicName>wrench</topicName>
+                    <updateRate>1000</updateRate>
+                    <gaussianNoise>0.0001</gaussianNoise>
+                </plugin>
+            </gazebo>
+            <xacro:if value="$(arg load_handle)">
+                <gazebo reference="handle_link">
+                    <material>Gazebo/White</material>
+                </gazebo>
+            </xacro:if>
+            <xacro:if value="$(arg load_calib_tool)">
+                <gazebo reference="calib_link">
+                    <material>Gazebo/White</material>
+                </gazebo>
+            </xacro:if>
+        </xacro:if>
+        <xacro:if value="$(arg load_model_joint_plugin)">
+            <gazebo>
+                <plugin name="model_joint_plugin" filename="libmodel_joint_plugin.so">
+                    <!-- <robotNamespace>~</robotNamespace> -->
+                    <topicName>~/$(arg robot_name)/joint_states</topicName>
+                    <numberOfStepsBeforeSync>10</numberOfStepsBeforeSync>
+                </plugin>
+            </gazebo>
+        </xacro:if>
+        <!-- The state publisher is done by the RTTStatePublisher() as on the real HW -->
+        <!--gazebo>
+        <plugin name="gz_state_pub" filename="libgazebo_ros_joint_state_publisher.so">
+        <jointName>joint_0,joint_1,joint_2,joint_3,joint_4,joint_5,joint_6</jointName>
+        <updateRate>100</updateRate>
+        <alwaysOn>true</alwaysOn>
+    </plugin>
+</gazebo-->
+<xacro:if value="$(arg load_base)">
+    <gazebo reference="base_link">
+        <material>Gazebo/Grey</material>
+    </gazebo>
+</xacro:if>
+<!-- base_link and link_0 are fixed, so merged by gazebo -->
+<xacro:unless value="$(arg load_base)">
+    <gazebo reference="base_link">
+        <material>Gazebo/Orange</material>
+    </gazebo>
+</xacro:unless>
+<xacro:gz_joint joint_name="joint_0"/>
+<xacro:gz_joint joint_name="joint_1"/>
+<xacro:gz_joint joint_name="joint_2"/>
+<xacro:gz_joint joint_name="joint_3"/>
+<xacro:gz_joint joint_name="joint_4"/>
+<xacro:gz_joint joint_name="joint_5"/>
+<xacro:gz_joint joint_name="joint_6"/>
+<xacro:enable_self_collision link_name="table_link"/>
+<!-- <xacro:enable_self_collision link_name="screwdriver_link"/>
+<xacro:enable_self_collision link_name="ati_link"/>
+<xacro:enable_self_collision link_name="link_7"/>
+<xacro:enable_self_collision link_name="head_cam_link"/>
+<xacro:enable_self_collision link_name="handle_link"/> -->
+<!-- If you want to add a Joint Torque sensor at each Joint -->
+<!--xacro:gz_ft_sensor joint_name="joint_0"/-->
+<!--xacro:gz_ft_sensor joint_name="joint_1"/-->
+<!--xacro:gz_ft_sensor joint_name="joint_2"/-->
+<!--xacro:gz_ft_sensor joint_name="joint_3"/-->
+<!--xacro:gz_ft_sensor joint_name="joint_4"/-->
+<!--xacro:gz_ft_sensor joint_name="joint_5"/-->
+<!--xacro:gz_ft_sensor joint_name="joint_6"/-->
+<gazebo reference="link_1">
+    <material>Gazebo/Orange</material>
+</gazebo>
+<gazebo reference="link_2">
+    <material>Gazebo/Orange</material>
+</gazebo>
+<gazebo reference="link_3">
+    <material>Gazebo/Orange</material>
+</gazebo>
+<gazebo reference="link_4">
+    <material>Gazebo/Orange</material>
+</gazebo>
+<gazebo reference="link_5">
+    <material>Gazebo/Orange</material>
+</gazebo>
+<gazebo reference="link_6">
+    <material>Gazebo/Grey</material>
+</gazebo>
+<gazebo reference="link_7">
+    <material>Gazebo/DarkGrey</material>
+</gazebo>
+</xacro:macro>
 </robot>

File: lwr_description/robots/kuka_lwr.urdf.xacro (robot description, xacro)
@@ -1,12 +1,19 @@
 <?xml version="1.0"?>
-<robot xmlns:xacro="http://www.ros.org/wiki/xacro"
+<robot xmlns:xacro="http://ros.org/wiki/xacro"
        name="lwr" >
-  <property name="M_PI" value="3.1415926535897931" />
-  <xacro:arg name="load_base" default="false"/>
+  <xacro:property name="M_PI" value="3.1415926535897931" />
+  <xacro:arg name="load_base" default="true"/>
   <xacro:arg name="load_ati_sensor" default="false"/>
   <xacro:arg name="load_calib_tool" default="false"/>
   <xacro:arg name="load_handle" default="false"/>
+  <xacro:arg name="load_hook" default="false"/>
+  <xacro:arg name="load_table" default="true"/>
+  <xacro:arg name="load_head_cam" default="false"/>
+  <xacro:arg name="load_screwdriver" default="false"/>
+  <xacro:arg name="robot_name" default="lwr"/>
   <!-- lwr-->
   <xacro:include filename="$(find lwr_description)/urdf/lwr.urdf.xacro" />
+  <!-- table-->
+  <xacro:include filename="$(find lwr_description)/urdf/table.urdf.xacro" />
   <!-- lwr_base -->
   <xacro:include filename="$(find lwr_description)/urdf/lwr_base.urdf.xacro" />
@@ -17,4 +24,10 @@
   <!-- handle -->
   <xacro:include filename="$(find lwr_description)/urdf/handle.urdf.xacro" />
+  <!-- hook -->
+  <xacro:include filename="$(find lwr_description)/urdf/hook.urdf.xacro" />
+  <!-- head_cam -->
+  <xacro:include filename="$(find lwr_description)/urdf/head_cam.urdf.xacro" />
+  <!-- screwdriver -->
+  <xacro:include filename="$(find lwr_description)/urdf/screwdriver.urdf.xacro" />
   <!-- generic simulator_gazebo plugins -->
   <xacro:include filename="$(find lwr_description)/gazebo/lwr.gazebo.urdf.xacro"/>
@@ -27,10 +40,17 @@
   <joint name="base_joint" type="fixed">
     <parent link="world"/>
-    <child link="base_link"/>
-    <origin xyz="0 0 0"/>
+    <xacro:if value="$(arg load_table)">
+      <child link="table_link"/>
+      <origin xyz="0 0 0.845"/>
+    </xacro:if>
+    <xacro:unless value="$(arg load_table)">
+      <child link="base_link"/>
+      <origin xyz="0 0 0.0"/>
+    </xacro:unless>
   </joint>
-  <xacro:lwr parent="base_link">
-    <origin xyz="0 0 0.02" rpy="0 0 ${2*M_PI/3}" />
-  </xacro:lwr>
+  <!-- table -->
+  <xacro:if value="$(arg load_table)">
+    <xacro:table/>
+  </xacro:if>
   <!-- lbr_base -->
   <xacro:if value="$(arg load_base)">
@@ -40,4 +60,8 @@
     <link name="base_link"/>
   </xacro:unless>
+  <!-- LWR -->
+  <xacro:lwr parent="base_link">
+    <origin xyz="0 0 0.02" rpy="0 0 ${2*M_PI/3}" />
+  </xacro:lwr>
   <!-- ati_sensor -->
   <xacro:if value="$(arg load_ati_sensor)">
@@ -51,4 +75,16 @@
       <xacro:handle/>
     </xacro:if>
+    <!-- hook -->
+    <xacro:if value="$(arg load_hook)">
+      <xacro:hook/>
+    </xacro:if>
+    <!-- head_cam -->
+    <xacro:if value="$(arg load_head_cam)">
+      <xacro:head_cam/>
+    </xacro:if>
+    <!-- screwdriver -->
+    <xacro:if value="$(arg load_screwdriver)">
+      <xacro:screwdriver/>
+    </xacro:if>
   </xacro:if>
    <xacro:lwr_gazebo/>

File: lwr_description/urdf/calib_tool.urdf.xacro (robot description, xacro)
@@ -1,4 +1,4 @@
 <?xml version="1.0" encoding="UTF-8"?>
-<robot xmlns:xacro="http://www.ros.org/wiki/xacro">
+<robot xmlns:xacro="http://ros.org/wiki/xacro">
    <xacro:macro name="calib_tool">
 	  <link name="calib_link">
@@ -38,4 +38,5 @@
 	    <parent link="ati_base_link" />
 	    <child link="calib_link" />
+        <limit effort="400" velocity="0" lower="0" upper="0" />
 	  </joint>
    </xacro:macro>

File: lwr_description/urdf/handle.urdf.xacro (robot description, xacro)
@@ -1,4 +1,4 @@
 <?xml version="1.0" encoding="UTF-8"?>
-<robot xmlns:xacro="http://www.ros.org/wiki/xacro">
+<robot xmlns:xacro="http://ros.org/wiki/xacro">
    <xacro:macro name="handle">
 	  <link name="handle_link">
@@ -38,4 +38,5 @@
 	    <parent link="ati_base_link" />
 	    <child link="handle_link" />
+        <limit effort="400" velocity="0" lower="0" upper="0" />
 	  </joint>
    </xacro:macro>
