Commit message: Update description for rtt_lwr-1.0

File: lwr_description/urdf/lwr.transmission.xacro (robot description, xacro)
@@ -2,74 +2,88 @@
 <robot xmlns:xacro="http://ros.org/wiki/xacro">
     <xacro:macro name="lwr_transmission">
-            <transmission name="trans_0">
-                        <type>transmission_interface/SimpleTransmission</type>
-                        <joint name="joint_0">
-				<hardwareInterface>EffortJointInterface</hardwareInterface>
-                        </joint>
-                        <actuator name="motor_0">
-                                <hardwareInterface>EffortJointInterface</hardwareInterface>
-                                <mechanicalReduction>1</mechanicalReduction>
-                        </actuator>
-            </transmission>
-                <transmission name="trans_1">
-                        <type>transmission_interface/SimpleTransmission</type>
-                        <joint name="joint_1">
-				<hardwareInterface>EffortJointInterface</hardwareInterface>
-                        </joint>
-                        <actuator name="motor_1">
-                                <hardwareInterface>EffortJointInterface</hardwareInterface>
-                                <mechanicalReduction>1</mechanicalReduction>
-                        </actuator>
-                </transmission>
-                <transmission name="trans_2">
-                        <type>transmission_interface/SimpleTransmission</type>
-                        <joint name="joint_2">
-				<hardwareInterface>EffortJointInterface</hardwareInterface>
-                        </joint>
-                        <actuator name="motor_2">
-                                <hardwareInterface>EffortJointInterface</hardwareInterface>
-                                <mechanicalReduction>1</mechanicalReduction>
-                        </actuator>
-                </transmission>
-                <transmission name="trans_3">
-                        <type>transmission_interface/SimpleTransmission</type>
-                        <joint name="joint_3">
-				<hardwareInterface>EffortJointInterface</hardwareInterface>
-                        </joint>
-                        <actuator name="motor_3">
-                                <hardwareInterface>EffortJointInterface</hardwareInterface>
-                                <mechanicalReduction>1</mechanicalReduction>
-                        </actuator>
-                </transmission>
-                <transmission name="trans_4">
-                        <type>transmission_interface/SimpleTransmission</type>
-                        <joint name="joint_4">
-				<hardwareInterface>EffortJointInterface</hardwareInterface>
-                        </joint>
-                        <actuator name="motor_4">
-                                <hardwareInterface>EffortJointInterface</hardwareInterface>
-                                <mechanicalReduction>1</mechanicalReduction>
-                        </actuator>
-                </transmission>
-                <transmission name="trans_5">
-                        <type>transmission_interface/SimpleTransmission</type>
-                        <joint name="joint_5">
-				<hardwareInterface>EffortJointInterface</hardwareInterface>
-                        </joint>
-                        <actuator name="motor_5">
-                                <hardwareInterface>EffortJointInterface</hardwareInterface>
-                                <mechanicalReduction>1</mechanicalReduction>
-                        </actuator>
-                </transmission>
-                <transmission name="trans_6">
-                        <type>transmission_interface/SimpleTransmission</type>
-                        <joint name="joint_6">
-				<hardwareInterface>EffortJointInterface</hardwareInterface>
-                        </joint>
-                        <actuator name="motor_6">
-                                <hardwareInterface>EffortJointInterface</hardwareInterface>
-                                <mechanicalReduction>1</mechanicalReduction>
-                        </actuator>
-                </transmission>
-        </xacro:macro>
+        <transmission name="trans_0">
+            <type>transmission_interface/SimpleTransmission</type>
+            <joint name="joint_0">
+                <hardwareInterface>EffortJointInterface</hardwareInterface>
+                <hardwareInterface>PositionJointInterface</hardwareInterface>
+            </joint>
+            <actuator name="motor_0">
+                <hardwareInterface>EffortJointInterface</hardwareInterface>
+                <hardwareInterface>PositionJointInterface</hardwareInterface>
+                <mechanicalReduction>1</mechanicalReduction>
+            </actuator>
+        </transmission>
+        <transmission name="trans_1">
+            <type>transmission_interface/SimpleTransmission</type>
+            <joint name="joint_1">
+                <hardwareInterface>EffortJointInterface</hardwareInterface>
+                <hardwareInterface>PositionJointInterface</hardwareInterface>
+            </joint>
+            <actuator name="motor_1">
+                <hardwareInterface>EffortJointInterface</hardwareInterface>
+                <hardwareInterface>PositionJointInterface</hardwareInterface>
+                <mechanicalReduction>1</mechanicalReduction>
+            </actuator>
+        </transmission>
+        <transmission name="trans_2">
+            <type>transmission_interface/SimpleTransmission</type>
+            <joint name="joint_2">
+                <hardwareInterface>EffortJointInterface</hardwareInterface>
+                <hardwareInterface>PositionJointInterface</hardwareInterface>
+            </joint>
+            <actuator name="motor_2">
+                <hardwareInterface>EffortJointInterface</hardwareInterface>
+                <hardwareInterface>PositionJointInterface</hardwareInterface>
+                <mechanicalReduction>1</mechanicalReduction>
+            </actuator>
+        </transmission>
+        <transmission name="trans_3">
+            <type>transmission_interface/SimpleTransmission</type>
+            <joint name="joint_3">
+                <hardwareInterface>EffortJointInterface</hardwareInterface>
+                <hardwareInterface>PositionJointInterface</hardwareInterface>
+            </joint>
+            <actuator name="motor_3">
+                <hardwareInterface>EffortJointInterface</hardwareInterface>
+                <hardwareInterface>PositionJointInterface</hardwareInterface>
+                <mechanicalReduction>1</mechanicalReduction>
+            </actuator>
+        </transmission>
+        <transmission name="trans_4">
+            <type>transmission_interface/SimpleTransmission</type>
+            <joint name="joint_4">
+                <hardwareInterface>EffortJointInterface</hardwareInterface>
+                <hardwareInterface>PositionJointInterface</hardwareInterface>
+            </joint>
+            <actuator name="motor_4">
+                <hardwareInterface>EffortJointInterface</hardwareInterface>
+                <hardwareInterface>PositionJointInterface</hardwareInterface>
+                <mechanicalReduction>1</mechanicalReduction>
+            </actuator>
+        </transmission>
+        <transmission name="trans_5">
+            <type>transmission_interface/SimpleTransmission</type>
+            <joint name="joint_5">
+                <hardwareInterface>EffortJointInterface</hardwareInterface>
+                <hardwareInterface>PositionJointInterface</hardwareInterface>
+            </joint>
+            <actuator name="motor_5">
+                <hardwareInterface>EffortJointInterface</hardwareInterface>
+                <hardwareInterface>PositionJointInterface</hardwareInterface>
+                <mechanicalReduction>1</mechanicalReduction>
+            </actuator>
+        </transmission>
+        <transmission name="trans_6">
+            <type>transmission_interface/SimpleTransmission</type>
+            <joint name="joint_6">
+                <hardwareInterface>EffortJointInterface</hardwareInterface>
+                <hardwareInterface>PositionJointInterface</hardwareInterface>
+            </joint>
+            <actuator name="motor_6">
+                <hardwareInterface>EffortJointInterface</hardwareInterface>
+                <hardwareInterface>PositionJointInterface</hardwareInterface>
+                <mechanicalReduction>1</mechanicalReduction>
+            </actuator>
+        </transmission>
+    </xacro:macro>
 </robot>

File: lwr_description/urdf/lwr.urdf.xacro (robot description, xacro)
@@ -1,26 +1,25 @@
 <?xml version="1.0" encoding="UTF-8"?>
-<robot xmlns:xacro="http://www.ros.org/wiki/xacro"
+<robot xmlns:xacro="http://ros.org/wiki/xacro"
       xmlns:controller="http://playerstage.sourceforge.net/gazebo/xmlschema/#controller"
    name="lwr" >
-   <xacro:property name="velocity_scale" value="50.0"/>
-   <xacro:property name="effort_scale" value="50.0"/>
+   <xacro:property name="velocity_scale" value="1.0"/>
+   <xacro:property name="effort_scale" value="10.0"/>
    <xacro:property name="M_PI" value="3.1415926535897931" />
-   <xacro:property name="damping_factor" value="0.2"/>
-   <xacro:property name="d0" value="${damping_factor*5.5}"/>
-   <xacro:property name="d1" value="${damping_factor*5.5}"/>
-   <xacro:property name="d2" value="${damping_factor*3.5}"/>
-   <xacro:property name="d3" value="${damping_factor*3.5}"/>
-   <xacro:property name="d4" value="${damping_factor*3.5}"/>
-   <xacro:property name="d5" value="${damping_factor*1.1}"/>
-   <xacro:property name="d6" value="${damping_factor*0.1}"/>
-   <xacro:property name="friction_factor" value="2.0"/>
+   <xacro:property name="damping_factor" value="0.1"/>
+   <xacro:property name="d0" value="${damping_factor*2.0}"/>
+   <xacro:property name="d1" value="${damping_factor*1.8}"/>
+   <xacro:property name="d2" value="${damping_factor*1.0}"/>
+   <xacro:property name="d3" value="${damping_factor*1.5}"/>
+   <xacro:property name="d4" value="${damping_factor*1.2}"/>
+   <xacro:property name="d5" value="${damping_factor*1.0}"/>
+   <xacro:property name="d6" value="${damping_factor*1.0}"/>
+   <xacro:property name="friction_factor" value="1.0"/>
    <xacro:property name="f0" value="${friction_factor*1.0}"/>
    <xacro:property name="f1" value="${friction_factor*1.0}"/>
    <xacro:property name="f2" value="${friction_factor*1.0}"/>
    <xacro:property name="f3" value="${friction_factor*1.0}"/>
-   <xacro:property name="f4" value="${friction_factor*1.0}"/>
-   <xacro:property name="f5" value="${friction_factor*1.0}"/>
-   <xacro:property name="f6" value="${friction_factor*1.0}"/>
-  <!-- Gazebo joint configuration -->
+   <xacro:property name="f4" value="${friction_factor*0.4}"/>
+   <xacro:property name="f5" value="${friction_factor*0.1}"/>
+   <xacro:property name="f6" value="${friction_factor*0.1}"/>
    <xacro:macro name="lwr" params="parent *origin ">
       <!-- joint between {parent} and lwr_0_link -->
@@ -38,10 +37,10 @@
               value="1.21032454350876" />
             <inertia
-              ixx="0.00262560565710656"
+              ixx="0.0262560565710656"
               ixy="-5.2754950052563E-07"
               ixz="3.77940202490646E-05"
-              iyy="0.00280724642508563"
+              iyy="0.0280724642508563"
               iyz="-2.56972470148208E-07"
-              izz="0.00306998250407766" />
+              izz="0.0306998250407766" />
           </inertial>
          <visual>
@@ -73,13 +72,13 @@
               xyz="-6.33965437334127E-08 0.0233273473346096 0.118146290406178"
               rpy="0 0 0" />
-            <mass
-              value="2.30339938771869" />
+              <mass
+                value="2.30339938771869" />
             <inertia
-              ixx="0.0156081163626041"
+              ixx="0.156081163626041"
               ixy="5.97319920503909E-08"
               ixz="-1.64780770629425E-07"
-              iyy="0.0153467542173805"
-              iyz="0.00319168949093809"
-              izz="0.00440736079943446" />
+              iyy="0.153467542173805"
+              iyz="0.0319168949093809"
+              izz="0.0440736079943446" />
           </inertial>
          <visual>
@@ -111,6 +110,6 @@
         xyz="1.26774962153076E-06 -0.032746486541291 0.0736556727355962"
         rpy="0 0 0" />
-      <mass
-        value="2.30343543179071" />
+        <mass
+          value="2.30343543179071" />
       <inertia
         ixx="0.0142348526057094"
@@ -157,6 +156,6 @@
         xyz="-1.40921289121243E-06 -0.0233297626126898 0.11815047247629"
         rpy="0 0 0" />
-      <mass
-        value="2.30342143971329" />
+        <mass
+          value="2.30342143971329" />
       <inertia
         ixx="0.0156098024078732"
@@ -195,6 +194,6 @@
         xyz="1.12239473548659E-07 0.0327442387470235 0.073658815701594"
         rpy="0 0 0" />
-      <mass
-        value="2.30343586527606" />
+        <mass
+          value="2.30343586527606" />
       <inertia
         ixx="0.0142336552604204"
@@ -233,6 +232,6 @@
         xyz="-6.00824789920296E-07 0.0207751869661564 0.0862053948486382"
         rpy="0 0 0" />
-      <mass
-        value="1.60059828363332" />
+        <mass
+          value="1.60059828363332" />
       <inertia
         ixx="0.00880806620496216"
@@ -271,13 +270,13 @@
         xyz="-2.64519244286276E-08 -0.00451753627467652 -0.00295324741635017"
         rpy="0 0 0" />
-      <mass
-        value="1.49302436988808" />
-      <inertia
-        ixx="0.00298541138330797"
-        ixy="-3.97658663154265E-09"
-        ixz="-1.71667243685877E-09"
-        iyy="0.00299834927882566"
-        iyz="-2.53647350791604E-05"
-        izz="0.00323627047307316" />
+        <mass
+          value="1.49302436988808" />
+        <inertia
+          ixx="0.0298541138330797"
+          ixy="-3.97658663154265E-09"
+          ixz="-1.71667243685877E-09"
+          iyy="0.0299834927882566"
+          iyz="-2.53647350791604E-05"
+          izz="0.0323627047307316" />
     </inertial>
          <visual>
@@ -309,13 +308,13 @@
         xyz="2.77555756156289E-17 1.11022302462516E-16 -0.015814675599801"
         rpy="0 0 0" />
-      <mass
-        value="0.108688241139613" />
-      <inertia
-        ixx="4.17908737998876E-05"
-        ixy="0"
-        ixz="0"
-        iyy="4.17908737998876E-05"
-        iyz="0"
-        izz="7.00756879151782E-05" />
+        <mass
+          value="0.108688241139613" />
+        <inertia
+          ixx="4.17908737998876E-02"
+          ixy="0"
+          ixz="0"
+          iyy="4.17908737998876E-02"
+          iyz="0"
+          izz="7.00756879151782E-02" />
     </inertial>
          <visual>
