Commit message: update ft sensor pos

File: lwr_description/robots/kuka_lwr.urdf.xacro (robot description, xacro)
@@ -22,9 +22,21 @@
   </gazebo>
   <xacro:macro name="tool">
-    <link name="ati_link"/>
+    <link name="ati_link">
+      <inertial>
+        <origin xyz="0 0 0" rpy="0 0 0" />
+        <mass value="0.730" />
+        <inertia
+          ixx="0.0001"
+          ixy="0.0"
+          ixz="0.0"
+          iyy="0.0001"
+          iyz="0.0"
+          izz="0.0001" />
+      </inertial>
+    </link>
     <joint name="ati_joint" type="fixed">
        <parent link="link_7" />
        <child link="ati_link" />
-       <origin xyz="0 0 0.049" rpy="0 0 0" />
+       <origin xyz="0 0 0.049" rpy="0 0 ${20.0*M_PI/180.0}" />
     </joint>
   </xacro:macro>

Commit message: add ati polaris link

File: lwr_description/robots/kuka_lwr.urdf.xacro (robot description, xacro)
@@ -38,5 +38,11 @@
        <parent link="link_7" />
        <child link="ati_link" />
-       <origin xyz="0 0 0.049" rpy="0 0 ${20.0*M_PI/180.0}" />
+       <origin xyz="0 0 0.0488" rpy="0 0 ${20.0*M_PI/180.0}" />
+    </joint>
+    <link name="ati_polaris_link"/>
+    <joint name="ati_polaris_joint" type="fixed">
+       <parent link="ati_link" />
+       <child link="ati_polaris_link" />
+       <origin xyz="0 0 0.0584" rpy="0 0 0" />
     </joint>
   </xacro:macro>

Commit message: ati sensor moved

File: lwr_description/robots/kuka_lwr.urdf.xacro (robot description, xacro)
@@ -44,5 +44,5 @@
        <parent link="ati_link" />
        <child link="ati_polaris_link" />
-       <origin xyz="0 0 0.0584" rpy="0 0 0" />
+       <origin xyz="0 0 0.0584" rpy="0 0 ${-M_PI/2}" />
     </joint>
   </xacro:macro>

Commit message: Adding new frame for calibration - Adding meshes

File: lwr_description/robots/kuka_lwr.urdf.xacro (robot description, xacro)
@@ -34,4 +34,17 @@
           izz="0.0001" />
       </inertial>
+      <visual>
+	<origin rpy="${M_PI/2.0} 0 ${20.0*M_PI/180.0}" xyz="0.0 0.0 -0.0388"/>
+	<geometry>
+	  <mesh filename="package://lwr_description/meshes/ati/ati.stl" scale="0.001 0.001 0.001"/>
+	</geometry>
+	<material name="color_j7"/>
+      </visual>
+      <collision>
+	<origin rpy="${M_PI/2.0} 0 ${20.0*M_PI/180.0}" xyz="0.0 0.0 -0.0388"/>
+	<geometry>
+	  <mesh filename="package://lwr_description/meshes/ati/ati.stl" scale="0.001 0.001 0.001"/>
+	</geometry>
+      </collision>
     </link>
     <joint name="ati_joint" type="fixed">
@@ -47,4 +60,32 @@
     </joint>
   </xacro:macro>
+  <!-- calib_tool -->
+  <link name="calib_link">
+    <visual>
+      <origin rpy="0 0 0" xyz="0.0 0.0 0"/>
+      <geometry>
+	<mesh filename="package://lwr_description/meshes/calib_tool/calib_tool.stl" scale="0.001 0.001 0.001"/>
+      </geometry>
+      <material name="color_j2"/>
+    </visual>
+    <collision>
+      <origin rpy="0 0 0" xyz="0.0 0.0 0"/>
+      <geometry>
+	<mesh filename="package://lwr_description/meshes/calib_tool/calib_tool.stl" scale="0.001 0.001 0.001"/>
+      </geometry>
+      <material name="color_j2"/>
+    </collision>
+  </link>
+  <joint name="ati_rot_joint" type="fixed">
+       <parent link="ati_link" />
+       <child link="ati_rot_link" />
+       <origin rpy="0 0 -${45.0*M_PI/180.0}" xyz="0 0 0"  />
+  </joint>
+  <link name="ati_rot_link"/>
+  <joint name="balls_joint" type="fixed">
+       <parent link="ati_rot_link" />
+       <child link="calib_link" />
+       <origin rpy="0 0 0" xyz="0.071 0 -0.0288"  />
+  </joint>
   <!--lbr-->
   <xacro:lwr parent="base_link">

Commit message: Adding new meshes into the urdf: lwr_base, handle, calib_tool Still needs collision files and roslaunch args

File: lwr_description/robots/kuka_lwr.urdf.xacro (robot description, xacro)
@@ -3,6 +3,18 @@
        name="lwr" >
   <property name="M_PI" value="3.1415926535897931" />
-  <!-- lbr-->
+  <property name="load_base" value="true" />
+  <property name="load_ati_sensor" value="true" />
+  <property name="load_calib_tool" value="true" />
+  <property name="load_handle" value="true" />
+  <!-- lwr-->
   <xacro:include filename="$(find lwr_description)/urdf/lwr.urdf.xacro" />
+  <!-- lwr_base -->
+  <xacro:include filename="$(find lwr_description)/urdf/lwr_base.urdf.xacro" />
+  <!-- ati_sensor -->
+  <xacro:include filename="$(find lwr_description)/urdf/ati_sensor.urdf.xacro" />
+  <!-- calib_tool -->
+  <xacro:include filename="$(find lwr_description)/urdf/calib_tool.urdf.xacro" />
+  <!-- handle -->
+  <xacro:include filename="$(find lwr_description)/urdf/handle.urdf.xacro" />
   <!-- generic simulator_gazebo plugins -->
   <xacro:include filename="$(find lwr_description)/gazebo/lwr.gazebo.urdf.xacro"/>
@@ -12,5 +24,5 @@
   <!-- world-->
   <link name="world"/>
-  <link name="base_link"/>
+  <!-- lbr -->
   <joint name="base_joint" type="fixed">
     <parent link="world"/>
@@ -18,78 +30,27 @@
     <origin xyz="0 0 0"/>
   </joint>
-  <xacro:macro name="tool">
-    <link name="ati_link">
-      <inertial>
-        <origin xyz="0 0 0" rpy="0 0 0" />
-        <mass value="0.730" />
-        <inertia
-          ixx="0.0001"
-          ixy="0.0"
-          ixz="0.0"
-          iyy="0.0001"
-          iyz="0.0"
-          izz="0.0001" />
-      </inertial>
-      <visual>
-	<origin rpy="${M_PI/2.0} 0 ${20.0*M_PI/180.0}" xyz="0.0 0.0 -0.0388"/>
-	<geometry>
-	  <mesh filename="package://lwr_description/meshes/ati/ati.stl" scale="0.001 0.001 0.001"/>
-	</geometry>
-	<material name="color_j7"/>
-      </visual>
-      <collision>
-	<origin rpy="${M_PI/2.0} 0 ${20.0*M_PI/180.0}" xyz="0.0 0.0 -0.0388"/>
-	<geometry>
-	  <mesh filename="package://lwr_description/meshes/ati/ati.stl" scale="0.001 0.001 0.001"/>
-	</geometry>
-      </collision>
-    </link>
-    <joint name="ati_joint" type="fixed">
-       <parent link="link_7" />
-       <child link="ati_link" />
-       <origin xyz="0 0 0.0488" rpy="0 0 ${20.0*M_PI/180.0}" />
-    </joint>
-    <link name="ati_polaris_link"/>
-    <joint name="ati_polaris_joint" type="fixed">
-       <parent link="ati_link" />
-       <child link="ati_polaris_link" />
-       <origin xyz="0 0 0.0584" rpy="0 0 ${-M_PI/2}" />
-    </joint>
-  </xacro:macro>
-  <!-- calib_tool -->
-  <link name="calib_link">
-    <visual>
-      <origin rpy="0 0 0" xyz="0.0 0.0 0"/>
-      <geometry>
-	<mesh filename="package://lwr_description/meshes/calib_tool/calib_tool.stl" scale="0.001 0.001 0.001"/>
-      </geometry>
-      <material name="color_j2"/>
-    </visual>
-    <collision>
-      <origin rpy="0 0 0" xyz="0.0 0.0 0"/>
-      <geometry>
-	<mesh filename="package://lwr_description/meshes/calib_tool/calib_tool.stl" scale="0.001 0.001 0.001"/>
-      </geometry>
-      <material name="color_j2"/>
-    </collision>
-  </link>
-  <joint name="ati_rot_joint" type="fixed">
-       <parent link="ati_link" />
-       <child link="ati_rot_link" />
-       <origin rpy="0 0 -${45.0*M_PI/180.0}" xyz="0 0 0"  />
-  </joint>
-  <link name="ati_rot_link"/>
-  <joint name="balls_joint" type="fixed">
-       <parent link="ati_rot_link" />
-       <child link="calib_link" />
-       <origin rpy="0 0 0" xyz="0.071 0 -0.0288"  />
-  </joint>
-  <!--lbr-->
   <xacro:lwr parent="base_link">
-    <!-- Position from origin -->
     <origin xyz="0 0 0.01" rpy="0 0 ${2*M_PI/3}" />
   </xacro:lwr>
+  <!-- lbr_base -->
+  <xacro:if value="${load_base}">
+    <xacro:lwr_base/>
+  </xacro:if>
+  <xacro:unless value="${load_base}">
+    <link name="base_link"/>
+  </xacro:unless>
+  <!-- ati_sensor -->
+  <xacro:if value="${load_ati_sensor}">
+    <xacro:ati_sensor/>
+    <!-- calib_tool -->
+    <xacro:if value="${load_calib_tool}">
+      <xacro:calib_tool/>
+    </xacro:if>
+    <!-- handle -->
+    <xacro:if value="${load_handle}">
+      <xacro:handle/>
+    </xacro:if>
+  </xacro:if>
    <xacro:lwr_gazebo/>
    <xacro:lwr_transmission/>
-   <xacro:tool/>
 </robot>

Commit message: fix base in gazebo

File: lwr_description/robots/kuka_lwr.urdf.xacro (robot description, xacro)
@@ -31,5 +31,5 @@
   </joint>
   <xacro:lwr parent="base_link">
-    <origin xyz="0 0 0.01" rpy="0 0 ${2*M_PI/3}" />
+    <origin xyz="0 0 0.02" rpy="0 0 ${2*M_PI/3}" />
   </xacro:lwr>
   <!-- lbr_base -->

File: lwr_description/urdf/lwr_base.urdf.xacro (robot description, xacro)
@@ -4,5 +4,5 @@
 	  <link name="base_link">
 	    <visual>
-	      <origin rpy="0 0 0" xyz="0 0 0"/>
+	      <origin rpy="0 0 0" xyz="0 0 0.01"/>
 	      <geometry>
 		<mesh filename="package://lwr_description/meshes/lwr_base/lwr_base.stl"/>
@@ -11,5 +11,5 @@
 	    </visual>
 	    <collision>
-	      <origin rpy="0 0 0" xyz="0 0 0"/>
+	      <origin rpy="0 0 0" xyz="0 0 0.01"/>
 	      <geometry>
 		<mesh filename="package://lwr_description/meshes/lwr_base/lwr_base_collision.stl"/>

Commit message: fix lwr base link

File: lwr_description/robots/kuka_lwr.urdf.xacro (robot description, xacro)
@@ -34,7 +34,4 @@
     <origin xyz="0 0 0"/>
   </joint>
-  <xacro:lwr parent="base_link">
-    <origin xyz="0 0 0.02" rpy="0 0 ${2*M_PI/3}" />
-  </xacro:lwr>
   <!-- lbr_base -->
   <xacro:if value="$(arg load_base)">
@@ -44,4 +41,8 @@
     <link name="base_link"/>
   </xacro:unless>
+  <!-- LWR -->
+  <xacro:lwr parent="base_link">
+    <origin xyz="0 0 0.02" rpy="0 0 ${2*M_PI/3}" />
+  </xacro:lwr>
   <!-- ati_sensor -->
   <xacro:if value="$(arg load_ati_sensor)">

Commit message: Add a table to the robot's description

File: lwr_description/robots/kuka_lwr.urdf.xacro (robot description, xacro)
@@ -8,7 +8,10 @@
   <xacro:arg name="load_handle" default="false"/>
   <xacro:arg name="load_hook" default="false"/>
+  <xacro:arg name="load_table" default="true"/>
   <xacro:arg name="robot_name" default="lwr"/>
   <!-- lwr-->
   <xacro:include filename="$(find lwr_description)/urdf/lwr.urdf.xacro" />
+  <!-- table-->
+  <xacro:include filename="$(find lwr_description)/urdf/table.urdf.xacro" />
   <!-- lwr_base -->
   <xacro:include filename="$(find lwr_description)/urdf/lwr_base.urdf.xacro" />
@@ -31,7 +34,17 @@
   <joint name="base_joint" type="fixed">
     <parent link="world"/>
-    <child link="base_link"/>
-    <origin xyz="0 0 0"/>
+    <xacro:if value="$(arg load_table)">
+      <child link="table_link"/>
+      <origin xyz="0 0 0.845"/>
+    </xacro:if>
+    <xacro:unless value="$(arg load_table)">
+      <child link="base_link"/>
+      <origin xyz="0 0 0.0"/>
+    </xacro:unless>
   </joint>
+  <!-- table -->
+  <xacro:if value="$(arg load_table)">
+    <xacro:table/>
+  </xacro:if>
   <!-- lbr_base -->
   <xacro:if value="$(arg load_base)">

Commit message: fix a few warnings on kinetic

File: lwr_description/robots/kuka_lwr.urdf.xacro (robot description, xacro)
@@ -1,6 +1,6 @@
 <?xml version="1.0"?>
-<robot xmlns:xacro="http://www.ros.org/wiki/xacro"
+<robot xmlns:xacro="http://ros.org/wiki/xacro"
        name="lwr" >
-  <property name="M_PI" value="3.1415926535897931" />
+  <xacro:property name="M_PI" value="3.1415926535897931" />
   <xacro:arg name="load_base" default="true"/>
   <xacro:arg name="load_ati_sensor" default="false"/>

File: lwr_description/urdf/ati_sensor.urdf.xacro (robot description, xacro)
@@ -1,4 +1,4 @@
 <?xml version="1.0" encoding="UTF-8"?>
-<robot xmlns:xacro="http://www.ros.org/wiki/xacro">
+<robot xmlns:xacro="http://ros.org/wiki/xacro">
    <xacro:macro name="ati_sensor">
 	  <joint name="ati_base_joint" type="fixed">

File: lwr_description/urdf/calib_tool.urdf.xacro (robot description, xacro)
@@ -1,4 +1,4 @@
 <?xml version="1.0" encoding="UTF-8"?>
-<robot xmlns:xacro="http://www.ros.org/wiki/xacro">
+<robot xmlns:xacro="http://ros.org/wiki/xacro">
    <xacro:macro name="calib_tool">
 	  <link name="calib_link">

File: lwr_description/urdf/handle.urdf.xacro (robot description, xacro)
@@ -1,4 +1,4 @@
 <?xml version="1.0" encoding="UTF-8"?>
-<robot xmlns:xacro="http://www.ros.org/wiki/xacro">
+<robot xmlns:xacro="http://ros.org/wiki/xacro">
    <xacro:macro name="handle">
 	  <link name="handle_link">

File: lwr_description/urdf/hook.urdf.xacro (robot description, xacro)
@@ -1,4 +1,4 @@
 <?xml version="1.0" encoding="UTF-8"?>
-<robot xmlns:xacro="http://www.ros.org/wiki/xacro">
+<robot xmlns:xacro="http://ros.org/wiki/xacro">
 	<xacro:macro name="hook">
   	<link name="hook_link">

File: lwr_description/urdf/lwr.urdf.xacro (robot description, xacro)
@@ -1,4 +1,4 @@
 <?xml version="1.0" encoding="UTF-8"?>
-<robot xmlns:xacro="http://www.ros.org/wiki/xacro"
+<robot xmlns:xacro="http://ros.org/wiki/xacro"
       xmlns:controller="http://playerstage.sourceforge.net/gazebo/xmlschema/#controller"
    name="lwr" >

File: lwr_description/urdf/lwr_base.urdf.xacro (robot description, xacro)
@@ -1,4 +1,4 @@
 <?xml version="1.0" encoding="UTF-8"?>
-<robot xmlns:xacro="http://www.ros.org/wiki/xacro">
+<robot xmlns:xacro="http://ros.org/wiki/xacro">
    <xacro:macro name="lwr_base">
 	  <link name="base_link">

File: lwr_description/urdf/table.urdf.xacro (robot description, xacro)
@@ -1,4 +1,4 @@
 <?xml version="1.0" encoding="UTF-8"?>
-<robot xmlns:xacro="http://www.ros.org/wiki/xacro">
+<robot xmlns:xacro="http://ros.org/wiki/xacro">
    <xacro:macro name="table">
 	  <link name="table_link">

Commit message: Adding screwdriver to the robot

File: lwr_description/robots/kuka_lwr.urdf.xacro (robot description, xacro)
@@ -10,4 +10,5 @@
   <xacro:arg name="load_table" default="true"/>
   <xacro:arg name="load_head_cam" default="true"/>
+  <xacro:arg name="load_screwdriver" default="true"/>
   <xacro:arg name="robot_name" default="lwr"/>
   <!-- lwr-->
@@ -27,4 +28,6 @@
   <!-- head_cam -->
   <xacro:include filename="$(find lwr_description)/urdf/head_cam.urdf.xacro" />
+  <!-- screwdriver -->
+  <xacro:include filename="$(find lwr_description)/urdf/screwdriver.urdf.xacro" />
   <!-- generic simulator_gazebo plugins -->
   <xacro:include filename="$(find lwr_description)/gazebo/lwr.gazebo.urdf.xacro"/>
@@ -80,4 +83,8 @@
       <xacro:head_cam/>
     </xacro:if>
+    <!-- screwdriver -->
+    <xacro:if value="$(arg load_screwdriver)">
+      <xacro:screwdriver/>
+    </xacro:if>
   </xacro:if>
    <xacro:lwr_gazebo/>

File: lwr_description/urdf/head_cam.urdf.xacro (robot description, xacro)
@@ -1,89 +1,41 @@
 <?xml version="1.0" encoding="UTF-8"?>
 <robot xmlns:xacro="http://www.ros.org/wiki/xacro">
-   <xacro:property name="epingle_length" value="0.09" />
-   <xacro:property name="epingle_radius" value="0.002" />
-   <xacro:property name="motor_length" value="0.02" />
-   <xacro:property name="motor_radius" value="0.025" />
-   <xacro:macro name="head_cam">
-     <link name="epingle_link" >
-       <inertial>
-         <origin xyz="0 0 0.5" rpy="0 0 0"/>
-         <mass value="0.1"/>
-         <inertia ixx="0.001"  ixy="0"  ixz="0" iyy="0.001" iyz="0" izz="0.001" />
-       </inertial>
-       <visual name="motor">
-         <origin xyz="0 0 0" rpy="0 0 0" />
-         <geometry>
-           <cylinder length="${motor_length}" radius="${motor_radius}" />
-         </geometry>
-       </visual>
-       <visual name="epingle">
-         <origin xyz="0 0 ${epingle_length/2.0}" rpy="0 0 0" />
-         <geometry>
-           <cylinder length="${epingle_length}" radius="${epingle_radius}" />
-         </geometry>
-       </visual>
-       <collision name="motor_collision">
-         <origin xyz="0 0 0" rpy="0 0 0" />
-         <geometry>
-           <cylinder length="${motor_length}" radius="${motor_radius}" />
-         </geometry>
-       </collision>
-       <collision name="epingle_collision">
-         <origin xyz="0 0 ${epingle_length/2.0}" rpy="0 0 0" />
-         <geometry>
-           <cylinder length="${epingle_length}" radius="${epingle_radius}" />
-         </geometry>
-      </collision>
-    </link>
-    <joint name="epingle_joint" type="fixed">
-      <origin xyz="0 0 ${motor_length/2.0}" rpy="0 0 0"/>
-      <parent link="ati_link"/>
-      <child link="epingle_link"/>
-    </joint>
-	  <link name="cam_link" >
+  <xacro:macro name="head_cam">
+    <link name="head_cam_link">
       <inertial>
-        <origin xyz="${-0.045/2.0} ${-0.042/2.0} ${-0.032/2.0}" rpy="0 0 0"/>
-        <mass value="0.1"/>
-        <inertia ixx="0.001"  ixy="0"  ixz="0" iyy="0.001" iyz="0" izz="0.001" />
+        <origin xyz="-0.001317 0.032906 -0.0621" rpy="0 0 0" />
+        <mass value="0.23396" />
+        <inertia
+          ixx="0.00047366"
+          ixy="-5.9303E-07"
+          ixz="1.6112E-06"
+          iyy="0.00016812"
+          iyz="-1.0497E-05"
+          izz="0.00043559" />
       </inertial>
       <visual>
-        <origin xyz="${-0.045/2.0} 0 0" rpy="0 0 0" />
+        <origin xyz="0 0 0" rpy="0 0 0" />
         <geometry>
-          <box size="0.045 0.042 0.032" />
+          <mesh filename="package://lwr_description/meshes/head_cam/head_cam.stl" />
         </geometry>
-        <material name="Cyan">
-          <color rgba="0 1.0 1.0 1.0"/>
+        <material name="">
+          <color rgba="0.49804 0.49804 0.49804 1" />
         </material>
       </visual>
       <collision>
-        <origin xyz="${-0.045/2.0} 0 0" rpy="0 0 0"/>
+        <origin xyz="0 0 0" rpy="0 0 0" />
         <geometry>
-          <box size="0.045 0.042 0.032" />
+          <mesh filename="package://lwr_description/meshes/head_cam/head_cam.stl" />
         </geometry>
       </collision>
-	  </link>
-    <link name="epingle_tip_link" />
-    <joint name="ati_to_tip_joint" type="fixed">
-      <origin rpy="${M_PI} 0 0" xyz="0 0 ${motor_length+epingle_length}" />
-	    <parent link="ati_link" />
-	    <child link="epingle_tip_link" />
-	  </joint>
-	  <joint name="ati_to_cam_joint" type="fixed">
-	    <!--origin rpy="${M_PI} ${-M_PI/2.0+atan(0.1/(motor_length+epingle_length))} ${M_PI}" xyz="0.1 0 0" /-->
-      	<origin rpy="${M_PI} -0.8329812666744316 ${M_PI}" xyz="0.1 0 0" />
-	    <parent link="ati_link" />
-	    <child link="cam_link" />
-	  </joint>
-    <link name="cam_link_optical" >
-	  </link>
-    <joint name="cam_optical_joint" type="fixed">
-      <!-- these values have to be these values otherwise the gazebo camera
-          image won't be aligned properly with the frame it is supposedly
-          originating from -->
-      <origin xyz="0 0 0" rpy="-1.570796 0 -1.570796"/>
-      <parent link="cam_link"/>
-      <child link="cam_link_optical"/>
+    </link>
+    <joint name="ati_to_cam_joint" type="fixed">
+        <origin
+          xyz="0.00138820343559641 -0.113248229330811 0.053096412734154"
+          rpy="-0.436332312998576 8.73838564895237E-16 3.05311331771918E-15" />
+        <parent link="ati_link" />
+        <child link="head_cam_link" />
+        <axis xyz="0 0 0" />
     </joint>
-   </xacro:macro>
+  </xacro:macro>
 </robot>

Commit message: add robot_description file as argument ability to load iiwa_descriptions

File: lwr_description/robots/kuka_lwr.urdf.xacro (robot description, xacro)
@@ -38,5 +38,5 @@
   <link name="world"/>
   <!-- lbr -->
-  <joint name="base_joint" type="fixed">
+  <joint name="world_joint" type="fixed">
     <parent link="world"/>
     <xacro:if value="$(arg load_table)">
